File: woodox/left_hand.kicad_sch (KiCad schematic)
At the start: 124 parts, among them IC2 W25Q16JVUXIQ_TR, IC3 IS31FL3741A-QFLS4-TR, J2 Conn_01x03_Female, J3 USB_C_Receptacle, J4 Interconnect Left, SW1 BOOT, SW2 RESET, U35 DRV5057A3, U36 DRV5057A3, U37 DRV5057A3, U38 DRV5057A3, U39 DRV5057A3, U40 DRV5057A3, U41 DRV5057A3, U42 DRV5057A3, U43 DRV5057A3, U44 CD74HC4067M, U45 DRV5057A3, U46 DRV5057A3, U47 DRV5057A3, U48 DRV5057A3, U49 DRV5057A3, U50 CD74HC4067M, U51 DRV5057A3, U52 DRV5057A3, U53 DRV5057A3, U54 DRV5057A3, U55 DRV5057A3, U56 DRV5057A3, U57 DRV5057A3, U58 DRV5057A3, U59 DRV5057A3, U60 DRV5057A3, U61 DRV5057A3, U62 DRV5057A3, U63 DRV5057A3, U64 DRV5057A3, U65 DRV5057A3, U66 DRV5057A3, U67 RP2040, U68 DRV5057A3, U69 DRV5057A3, U70 NCP1117-3.3_SOT223, Y1 ABLS-12.000MHZ-B4-T

Commit message: whatever the fuck i all did
Parts:
- removed C10, C11, C23, C25, C27: 1uF, Capacitor_SMD:C_0402_1005Metric, symbol Device:C_Small
- removed C12, C17: 10uF, Capacitor_SMD:C_0402_1005Metric, symbol pspice:CAP
- removed C13, C14, C15, C16, C18, C19, C20, C21, C22, C24, C26, C28, C7: 0.1uF, Capacitor_SMD:C_0402_1005Metric, symbol Device:C_Small
- removed C8, C9: 27pF, Capacitor_SMD:C_0402_1005Metric, symbol Device:C_Small
- removed D33, D34, D35, D36, D37, D38, D39, D40, D41, D42, D43, D44, D45, D46, D47, D48, D49, D50, D51, D52, D53, D54, D55, D56, D57, D58, D59, D60, D61, D62, D63, D64: LED_RGB, marbastlib-mx:LED_MX_6028R, symbol marbastlib-various:LED_6028R
- removed IC2: W25Q16JVUXIQ_TR, W25Q16JVUXIQ_TR:SON50P300X200X60-9N, symbol W25Q16JVUXIQ_TR:W25Q16JVUXIQ_TR
- removed IC3: IS31FL3741A-QFLS4-TR, IS31FL3741A-QFLS4-TR:QFN40P700X700X80-61N-D, symbol IS31FL3741A-QFLS4-TR:IS31FL3741A-QFLS4-TR
- removed J2: Conn_01x03_Female, Connector_PinHeader_2.54mm:PinHeader_1x03_P2.54mm_Vertical, symbol Connector:Conn_01x04_Female
- removed J3: USB_C_Receptacle, Connector_USB:USB_C_Receptacle_Amphenol_12401610E4-2A, symbol Connector:USB_C_Receptacle
- removed R19, R43, R44: 1k, Resistor_SMD:R_0603_1608Metric, symbol Device:R
- removed R20, R42: 10k, Resistor_SMD:R_0603_1608Metric, symbol Device:R
- removed R21, R22: 27.4, Resistor_SMD:R_0603_1608Metric, symbol Device:R
- removed R23, R24: 5k1, Resistor_SMD:R_0603_1608Metric, symbol Device:R
- removed R25, R27, R28, R30, R31, R33, R34, R35, R37, R38: 20, Resistor_SMD:R_0603_1608Metric, symbol Device:R
- removed R26, R29, R32, R36, R39: 51, Resistor_SMD:R_0603_1608Metric, symbol Device:R
- removed R40, R41: 2k, Resistor_SMD:R_0603_1608Metric, symbol Device:R
- removed SW1: BOOT, Button_Switch_SMD:SW_Push_1P1T_NO_6x6mm_H9.5mm, symbol Switch:SW_Push
- removed SW2: RESET, Button_Switch_SMD:SW_Push_1P1T_NO_6x6mm_H9.5mm, symbol Switch:SW_Push
- removed U50: CD74HC4067M, Package_SO:SOIC-24W_7.5x15.4mm_P1.27mm, symbol 74xx:CD74HC4067M
- removed U67: RP2040, Package_DFN_QFN:QFN-56-1EP_7x7mm_P0.4mm_EP3.2x3.2mm, symbol MCU_RaspberryPi:RP2040
- removed U70: NCP1117-3.3_SOT223, Package_TO_SOT_SMD:SOT-223-3_TabPin2, symbol Regulator_Linear:NCP1117-3.3_SOT223
- removed Y1: ABLS-12.000MHZ-B4-T, Crystal:Crystal_SMD_5032-2Pin_5.0x3.2mm, symbol Device:Crystal
- added C29, C35, C37: 0.1uF, Capacitor_SMD:C_0603_1608Metric, symbol Device:C_Small
- added C30, C31: 27pF, Capacitor_SMD:C_0603_1608Metric, symbol Device:C_Small
- added C32, C33, C36: 1uF, Capacitor_SMD:C_0603_1608Metric, symbol Device:C_Small
- added C34, C38: 10uF, Capacitor_SMD:C_0603_1608Metric, symbol pspice:CAP
- added IC4: W25Q16JVUXIQ_TR, W25Q16JVUXIQ_TR:SON50P300X200X60-9N, symbol W25Q16JVUXIQ_TR:W25Q16JVUXIQ_TR
- added J5: Conn_01x03_Female, Connector_PinHeader_2.54mm:PinHeader_1x04_P2.54mm_Vertical, symbol Connector:Conn_01x04_Female
- added J6: USB_C_Receptacle, Connector_USB:USB_C_Receptacle_Amphenol_12401610E4-2A, symbol Connector:USB_C_Receptacle
- added LED10, LED11, LED12, LED13, LED14, LED15, LED16, LED17, LED18, LED19, LED2, LED20, LED21, LED22, LED23, LED24, LED25, LED26, LED27, LED28, LED29, LED3, LED30, LED31, LED32, LED33, LED4, LED5, LED6, LED7, LED8, LED9: MX_SK6812MINI-E, lib:LED_MX_SK6812MINI-R, symbol marbastlib-mx:MX_SK6812MINI-E
- added R45, R47, R52: 1k, Resistor_SMD:R_0603_1608Metric, symbol Device:R
- added R46: 10k, Resistor_SMD:R_0603_1608Metric, symbol Device:R
- added R48, R49: 27.4, Resistor_SMD:R_0603_1608Metric, symbol Device:R
- added R50, R51: 5k1, Resistor_SMD:R_0603_1608Metric, symbol Device:R
- added SW3: BOOT, Button_Switch_SMD:SW_Push_1P1T_NO_Vertical_Wuerth_434133025816, symbol Switch:SW_Push
- added SW4: RESET, Button_Switch_SMD:SW_Push_1P1T_NO_Vertical_Wuerth_434133025816, symbol Switch:SW_Push
- added U50: RP2040, Package_DFN_QFN:QFN-56-1EP_7x7mm_P0.4mm_EP3.2x3.2mm, symbol MCU_RaspberryPi:RP2040
- added U71: CD74HC4067SM96E4, Package_SO:SSOP-24_5.3x8.2mm_P0.65mm, symbol 74xx:CD74HC4067M
- added U72: OLED_256x64_I2C, lib:OLED_256x64_I2C, symbol oled_256x64_i2c:OLED_256x64_I2C
- added U73: NCP1117-3.3_SOT223, Package_TO_SOT_SMD:SOT-223-3_TabPin2, symbol Regulator_Linear:NCP1117-3.3_SOT223
- added Y2: ECS-120-8-30-JGN-TR, Crystal:Crystal_SMD_5032-2Pin_5.0x3.2mm, symbol Device:Crystal
- U44: value CD74HC4067M -> CD74HC4067SM96E4; footprint Package_SO:SOIC-24W_7.5x15.4mm_P1.27mm -> Package_SO:SSOP-24_5.3x8.2mm_P0.65mm; MPN (none) -> CD74HC4067SM96E4
Connections:
- net I2C SCL is gone; now on net LED_USB: J4.B7 (D-)
- net MUX3 S0 is gone; now on net MUX S0: J4.A2 (TX1+)
- net MUX3 S1 is gone; now on net MUX S1: J4.A3 (TX1-)
- net MUX3 S2 is gone; now on net MUX S2: J4.B11 (RX1+)
- net MUX3 S3 is gone; now on net MUX S3: J4.B10 (RX1-)
- net MUX4 S0 is gone; now on net MUX S0: J4.B2 (TX2+)
- net MUX4 S1 is gone; now on net MUX S1: J4.B3 (TX2-)
- net MUX4 S2 is gone; now on net MUX S2: J4.A11 (RX2+)
- net MUX4 S3 is gone; now on net MUX S3: J4.A10 (RX2-)
- net +3.3V: now also U44.12 (GND), C29.1, C32.1, C36.1, C38.1, IC4.8 (VCC), J5.1 (Pin_1), R46.2, U50.1 (IOVDD), U50.10 (IOVDD), U50.22 (IOVDD), U50.33 (IOVDD), U50.42 (IOVDD), U50.43 (ADC_AVDD), U50.44 (VREG_IN), U50.48 (USB_VDD), U50.49 (IOVDD), U71.24 (VCC), U72.2 (VCC), U73.2 (VO); no longer J4.A4 (VBUS), J4.A9 (VBUS), J4.B4 (VBUS), J4.B9 (VBUS), U44.24 (VCC)
- net GND: now also U44.1 (COM), U44.24 (VCC), C29.2, C32.2, C33.1, C34.2, C35.1, C36.2, C37.1, C38.2, IC4.4 (GND), IC4.9 (EP), J5.4 (Pin_4), J6.A1 (GND), J6.A12 (GND), J6.B1 (GND), J6.B12 (GND), LED10.4 (VSS), LED11.4 (VSS), LED12.4 (VSS), LED13.4 (VSS), LED14.4 (VSS), LED15.4 (VSS), LED16.4 (VSS), LED17.4 (VSS), LED18.4 (VSS), LED19.4 (VSS), LED2.4 (VSS), LED20.4 (VSS), LED21.4 (VSS), LED22.4 (VSS), LED23.4 (VSS), LED24.4 (VSS), LED25.4 (VSS), LED26.4 (VSS), LED28.4 (VSS), LED29.4 (VSS), LED3.4 (VSS), LED30.4 (VSS), LED4.4 (VSS), LED5.4 (VSS), LED6.4 (VSS), LED7.4 (VSS), LED8.4 (VSS), LED9.4 (VSS), R50.2, R51.2, SW3.1, SW4.1, U50.19 (TESTEN), U50.57 (GND), U71.12 (GND), U71.15 (~{E}), U72.1 (GND), U73.1 (GND); no longer U44.12 (GND), U44.15 (~{E})
- net MUX1 COM: now also U44.15 (~{E}), U50.38 (GPIO26_ADC0); no longer U44.1 (COM)
- net MUX2 COM: now also U50.39 (GPIO27_ADC1), U71.1 (COM)
- net MUX3 COM: now also U50.40 (GPIO28_ADC2)
- net MUX4 COM: now also U50.41 (GPIO29_ADC3)
- net QSPI_SCLK: now also IC4.6 (CLK), U50.52 (QSPI_SCLK)
- net QSPI_SD0: now also IC4.5 (DI(IO0)), U50.53 (QSPI_SD0)
- net QSPI_SD1: now also IC4.2 (DO(IO1)), U50.55 (QSPI_SD1)
- net QSPI_SD2: now also IC4.3 (IO2), U50.54 (QSPI_SD2)
- net QSPI_SD3: now also IC4.7 (IO3), U50.51 (QSPI_SD3)
- net QSPI_SS: now also IC4.1 (~{CS}), R45.2, R46.1, U50.56 (QSPI_SS)
- net SENS1: now reaches J4.A5 (CC1)
- net LED_USB: now reaches J4.A7 (D-)
- net LED_USB: now also LED33.2 (DOUT)
- net SENS2: now reaches J4.B5 (CC2)
- net at U39.2 (OUT): now also U44.9 (I0); no longer U44.16 (I15)
- net at U43.2 (OUT): now also U44.4 (I5); no longer U44.21 (I10)
- net at U51.2 (OUT): now also U71.7 (I2)
- net at U49.2 (OUT): now also U44.22 (I9); no longer U44.3 (I6)
- net at U66.2 (OUT): now also U71.19 (I12)
- net at U38.2 (OUT): now also U44.8 (I1); no longer U44.17 (I14)
- net at U37.2 (OUT): now also U44.7 (I2); no longer U44.18 (I13)
- net at U64.2 (OUT): now also U71.23 (I8)
- net at U47.2 (OUT): now also U44.20 (I11); no longer U44.5 (I4)
- net at U58.2 (OUT): now also U71.4 (I5)
- net at U68.2 (OUT): now also U71.16 (I15)
- net at U69.2 (OUT): now also U71.17 (I14)
- net at U65.2 (OUT): now also U71.18 (I13)
- net at U56.2 (OUT): now also U71.2 (I7)
- net at U61.2 (OUT): now also U71.20 (I11)
- net at U62.2 (OUT): now also U71.21 (I10)
- net at U63.2 (OUT): now also U71.22 (I9)
- net at U57.2 (OUT): now also U71.3 (I6)
- net at U59.2 (OUT): now also U71.5 (I4)
- net at U60.2 (OUT): now also U71.6 (I3)
- net at U52.2 (OUT): now also U71.8 (I1)
- net at U53.2 (OUT): now also U71.9 (I0)
- net at U36.2 (OUT): now also U44.6 (I3); no longer U44.19 (I12)
- net at U45.2 (OUT): now also U44.18 (I13); no longer U44.7 (I2)
- net at U46.2 (OUT): now also U44.19 (I12); no longer U44.6 (I3)
- net at U54.2 (OUT): now also U44.16 (I15); no longer U44.9 (I0)
- net at U48.2 (OUT): now also U44.21 (I10); no longer U44.4 (I5)
- net at U35.2 (OUT): now also U44.5 (I4); no longer U44.20 (I11)
- net at U55.2 (OUT): now also U44.17 (I14); no longer U44.8 (I1)
- net at U41.2 (OUT): now also U44.2 (I7); no longer U44.23 (I8)
- net at U40.2 (OUT): now also U44.23 (I8); no longer U44.2 (I7)
- net at U42.2 (OUT): now also U44.3 (I6); no longer U44.22 (I9)
- net I2C SDA: no longer names the net of J4.B6 (D+)
- net MUX1 S0 renamed MUX S3
- net MUX S3: now also U50.6 (GPIO4), U71.10 (S0)
- net MUX1 S1 renamed MUX S2
- net MUX S2: now also U50.5 (GPIO3), U71.11 (S1)
- net MUX1 S2 renamed MUX S1
- net MUX S1: now also U50.4 (GPIO2), U71.14 (S2)
- net MUX1 S3 renamed MUX S0
- net MUX S0: now also U50.3 (GPIO1), U71.13 (S3)
- new net: LED27.3 (DIN), LED30.2 (DOUT)
- new net: LED29.2 (DOUT), LED30.3 (DIN)
- new net: LED21.2 (DOUT), LED22.3 (DIN)
- new net: LED20.2 (DOUT), LED21.3 (DIN)
- new net: LED6.2 (DOUT), LED7.3 (DIN)
- new net: LED5.2 (DOUT), LED6.3 (DIN)
- new net: LED27.2 (DOUT), LED31.3 (DIN)
- new net: LED27.4 (VSS), LED31.4 (VSS), LED32.4 (VSS), LED33.4 (VSS)
- new net: R52.1, SW4.2
- new net: LED15.2 (DOUT), LED16.3 (DIN)
- new net: LED14.2 (DOUT), LED15.3 (DIN)
- new net: LED12.2 (DOUT), LED13.3 (DIN)
- new net: LED11.2 (DOUT), LED12.3 (DIN)
- new net: J6.A6 (D+), J6.B6 (D+), R49.1
- new net: R49.2, U50.47 (USB_DP)
- new net: LED8.2 (DOUT), LED9.3 (DIN)
- new net: LED7.2 (DOUT), LED8.3 (DIN)
- new net: C33.2, C35.2, C37.2, U50.23 (DVDD), U50.45 (VREG_VOUT), U50.50 (DVDD)
- new net: LED13.2 (DOUT), LED14.3 (DIN)
- new net: C30.1, Y2.1
- new net: C30.2, R47.1
- new net: C31.1, Y2.2
- new net: LED19.2 (DOUT), LED20.3 (DIN)
- new net: LED17.2 (DOUT), LED18.3 (DIN)
- new net: LED16.2 (DOUT), LED17.3 (DIN)
- new net: LED26.2 (DOUT), LED28.3 (DIN)
- new net: LED25.2 (DOUT), LED26.3 (DIN)
- new net: LED4.2 (DOUT), LED5.3 (DIN)
- new net: R45.1, SW3.2
- new net: LED23.2 (DOUT), LED24.3 (DIN)
- new net: LED22.2 (DOUT), LED23.3 (DIN)
- new net: LED24.2 (DOUT), LED25.3 (DIN)
- new net: C31.2, U50.20 (XIN)
- new net: LED10.2 (DOUT), LED11.3 (DIN)
- new net: LED28.2 (DOUT), LED29.3 (DIN)
- new net: J6.A5 (CC1), R51.1
- new net: J6.A7 (D-), J6.B7 (D-), R48.1
- new net: J6.B5 (CC2), R50.1
- new net: LED32.2 (DOUT), LED33.3 (DIN)
- new net: LED31.2 (DOUT), LED32.3 (DIN)
- new net: LED3.2 (DOUT), LED4.3 (DIN)
- new net: LED2.2 (DOUT), LED3.3 (DIN)
- new net: LED10.3 (DIN), LED9.2 (DOUT)
- new net: R47.2, U50.21 (XOUT)
- new net: LED18.2 (DOUT), LED19.3 (DIN)
- new net: J5.2 (Pin_2), U50.25 (SWD)
- new net: J5.3 (Pin_3), U50.24 (SWCLK)
- new net: R52.2, U50.26 (RUN)
- new net: R48.2, U50.46 (USB_DM)
- new net +5V: C34.1, J4.A4 (VBUS), J4.A9 (VBUS), J4.B4 (VBUS), J4.B9 (VBUS), J6.A4 (VBUS), J6.A9 (VBUS), J6.B4 (VBUS), J6.B9 (VBUS), LED10.1 (VDD), LED11.1 (VDD), LED12.1 (VDD), LED13.1 (VDD), LED14.1 (VDD), LED15.1 (VDD), LED16.1 (VDD), LED17.1 (VDD), LED18.1 (VDD), LED19.1 (VDD), LED2.1 (VDD), LED20.1 (VDD), LED21.1 (VDD), LED22.1 (VDD), LED23.1 (VDD), LED24.1 (VDD), LED25.1 (VDD), LED26.1 (VDD), LED27.1 (VDD), LED28.1 (VDD), LED29.1 (VDD), LED3.1 (VDD), LED30.1 (VDD), LED31.1 (VDD), LED32.1 (VDD), LED33.1 (VDD), LED4.1 (VDD), LED5.1 (VDD), LED6.1 (VDD), LED7.1 (VDD), LED8.1 (VDD), LED9.1 (VDD), U73.3 (VI)
- new net D_CS: U50.12 (GPIO9), U72.7 (CS)
- new net D_DC: U50.13 (GPIO10), U72.6 (DC)
- new net D_RST: U50.14 (GPIO11), U72.5 (RST)
- new net D_SCL: U50.16 (GPIO13), U72.3 (SCL)
- new net D_SDA: U50.15 (GPIO12), U72.4 (SDA)
- new net LED: LED2.3 (DIN), U50.7 (GPIO5)
Other:
- moved on the sheet: J4

Commit message: redox woodox left hand pcb
Parts:
- removed J4: Interconnect Left, Connector_USB:USB_C_Receptacle_Amphenol_12401610E4-2A, symbol Connector:USB_C_Receptacle
- removed U44, U71: CD74HC4067SM96E4, Package_SO:SSOP-24_5.3x8.2mm_P0.65mm, symbol 74xx:CD74HC4067M
- added U71, U72, U73, U74: 74HC4051, Package_SO:TSSOP-16_4.4x5mm_P0.65mm, symbol 74xx:74HC4051
- renumbered C29 to C13, C30 to C14, C31 to C15, C32 to C16, C33 to C17, C34 to C18, C35 to C19, C36 to C20, C37 to C21, C38 to C22, IC4 to IC2, J5 to J4, J6 to J5, LED2 to LED33, LED13 to LED34, LED14 to LED35, LED25 to LED36, LED26 to LED37, LED3 to LED38, LED12 to LED39, LED15 to LED40, LED24 to LED41, LED4 to LED42, LED11 to LED43, LED16 to LED44, LED23 to LED45, LED28 to LED46, LED5 to LED47, LED10 to LED48, LED17 to LED49, LED22 to LED50, LED29 to LED51, LED6 to LED52, LED9 to LED53, LED18 to LED54, LED21 to LED55, LED30 to LED56, LED7 to LED57, LED8 to LED58, LED19 to LED59, LED20 to LED60, LED27 to LED61, LED33 to LED62, LED31 to LED63, LED32 to LED64, R46 to R10, R47 to R11, R48 to R12, R49 to R13, R50 to R14, R51 to R15, R52 to R16, R45 to R9, U36 to U38, U37 to U39, U38 to U40, U39 to U41, U35 to U42, U40 to U43, U41 to U44, U42 to U45, U43 to U46, U72 to U47, U45 to U48, U46 to U49, U47 to U50, U48 to U51, U49 to U52, U51 to U53, U52 to U54, U53 to U55, U54 to U56, U55 to U57, U56 to U58, U57 to U59, U58 to U60, U59 to U61, U50 to U62, U60 to U63, U61 to U64, U62 to U65, U63 to U66, U64 to U67, U65 to U68, U66 to U69, U73 to U70, U68 to U75, U69 to U76
Connections:
- net +3.3V: now also U71.16 (VCC), U72.16 (VCC), U73.16 (VCC), U74.16 (VCC); no longer C13.1, C16.1, IC2.8 (VCC), R10.2, U62.43 (ADC_AVDD), U62.44 (VREG_IN), U62.48 (USB_VDD)
- net +5V: no longer C18.1, LED33.1 (VDD), LED34.1 (VDD), LED35.1 (VDD), LED36.1 (VDD), LED37.1 (VDD), LED38.1 (VDD), LED39.1 (VDD), LED40.1 (VDD), LED41.1 (VDD), LED42.1 (VDD), LED43.1 (VDD), LED44.1 (VDD), LED45.1 (VDD), LED46.1 (VDD), LED47.1 (VDD), LED48.1 (VDD), LED49.1 (VDD), LED50.1 (VDD), LED51.1 (VDD), LED52.1 (VDD), LED53.1 (VDD), LED54.1 (VDD), LED55.1 (VDD), LED56.1 (VDD), LED57.1 (VDD), LED58.1 (VDD), LED59.1 (VDD), LED60.1 (VDD), LED61.1 (VDD), LED62.1 (VDD), LED63.1 (VDD), LED64.1 (VDD)
- net GND: now also U71.7 (VEE), U71.8 (GND), U72.7 (VEE), U72.8 (GND), U73.7 (VEE), U73.8 (GND), U74.7 (VEE), U74.8 (GND); no longer LED35.4 (VSS), LED36.4 (VSS), LED37.4 (VSS), LED40.4 (VSS), LED41.4 (VSS), LED44.4 (VSS), LED45.4 (VSS), LED46.4 (VSS), LED49.4 (VSS), LED50.4 (VSS), LED51.4 (VSS), LED54.4 (VSS), LED55.4 (VSS), LED56.4 (VSS), LED59.4 (VSS), LED60.4 (VSS), R14.2, R15.2
- net MUX S0: now also U71.11 (S0), U72.11 (S0), U73.11 (S0), U74.11 (S0)
- net MUX S1: now also U71.10 (S1), U72.10 (S1), U73.10 (S1), U74.10 (S1)
- net MUX S2: now also U71.9 (S2), U72.9 (S2), U73.9 (S2), U74.9 (S2)
- net MUX1 COM: now also U71.3 (A)
- net MUX2 COM: now also U72.3 (A)
- net MUX3 COM: now also U73.3 (A)
- net MUX4 COM: now also U74.3 (A)
- net at U41.2 (OUT): now also U71.14 (A1)
- net at U75.2 (OUT): now also U74.13 (A0)
- net at U76.2 (OUT): now also U73.13 (A0)
- net at U68.2 (OUT): now also U71.13 (A0)
- net at U69.2 (OUT): now also U72.13 (A0)
- net at U58.2 (OUT): now also U71.12 (A3)
- net at U64.2 (OUT): now also U71.15 (A2)
- net at U65.2 (OUT): now also U72.15 (A2)
- net at U66.2 (OUT): now also U73.15 (A2)
- net at U67.2 (OUT): now also U74.15 (A2)
- net at U59.2 (OUT): now also U72.12 (A3)
- net at U60.2 (OUT): now also U73.12 (A3)
- net at U61.2 (OUT): now also U74.12 (A3)
- net at U63.2 (OUT): now also U74.14 (A1)
- net at U53.2 (OUT): now also U71.1 (A4)
- net at U54.2 (OUT): now also U72.1 (A4)
- net at U55.2 (OUT): now also U73.1 (A4)
- net at U46.2 (OUT): now also U74.2 (A6)
- net at U52.2 (OUT): now also U72.14 (A1)
- net at J5.B6 (D+), R13.1: no longer J5.A6 (D+)
- net at C17.2, U62.23 (DVDD), U62.50 (DVDD): no longer C19.2, C21.2, U62.45 (VREG_VOUT)
- net at U40.2 (OUT): now also U74.4 (A7)
- net at U39.2 (OUT): now also U73.4 (A7)
- net at U50.2 (OUT): now also U73.5 (A5)
- net at C15.2: no longer U62.20 (XIN)
- net at J5.A7 (D-), J5.B7 (D-): no longer R12.1
- net at U38.2 (OUT): now also U72.4 (A7)
- net at U48.2 (OUT): now also U71.5 (A5)
- net at U49.2 (OUT): now also U72.5 (A5)
- net at U56.2 (OUT): now also U74.1 (A4)
- net at U57.2 (OUT): now also U73.14 (A1)
- net at U44.2 (OUT): now also U72.2 (A6)
- net at U51.2 (OUT): now also U74.5 (A5)
- net at U43.2 (OUT): now also U71.2 (A6)
- net at U45.2 (OUT): now also U73.2 (A6)
- net at U42.2 (OUT): now also U71.4 (A7)
- net MUX S3 renamed MUX E
- net MUX E: now also U71.6 (~{E}), U72.6 (~{E}), U73.6 (~{E}), U74.6 (~{E})
- new net: LED36.1 (VDD), LED37.1 (VDD), LED45.1 (VDD), LED46.1 (VDD), LED50.1 (VDD), LED51.1 (VDD), LED55.1 (VDD), LED56.1 (VDD), LED62.1 (VDD)
- new net: LED35.4 (VSS), LED36.4 (VSS), LED40.4 (VSS), LED41.4 (VSS), LED44.4 (VSS), LED45.4 (VSS), LED49.4 (VSS), LED50.4 (VSS), LED54.4 (VSS), LED55.4 (VSS), LED59.4 (VSS), LED60.4 (VSS)
- new net: IC2.8 (VCC), R10.2
- new net: LED34.1 (VDD), LED35.1 (VDD), LED39.1 (VDD), LED40.1 (VDD), LED43.1 (VDD), LED44.1 (VDD), LED48.1 (VDD), LED49.1 (VDD), LED53.1 (VDD), LED54.1 (VDD), LED58.1 (VDD), LED59.1 (VDD)
- new net: C16.1, U62.44 (VREG_IN)
- new net: R14.2, R15.2
- new net: C21.2, U62.45 (VREG_VOUT)
Other:
- moved on the sheet: U38, U39, U40, U41, U42, U43, U44, U45, U46, U48, U49, U50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
