File: woodox/right_hand.kicad_sch (KiCad schematic)
At the start: 92 parts, among them IC1 IS31FL3741A-QFLS4-TR, J1 USB_C_Receptacle, U1 DRV5057A3, U10 DRV5057A3, U11 DRV5057A3, U12 DRV5057A3, U13 DRV5057A3, U14 DRV5057A3, U15 DRV5057A3, U16 DRV5057A3, U17 DRV5057A3, U18 DRV5057A3, U19 DRV5057A3, U2 DRV5057A3, U20 DRV5057A3, U21 DRV5057A3, U22 DRV5057A3, U23 DRV5057A3, U24 CD74HC4067M, U25 CD74HC4067M, U26 DRV5057A3, U27 DRV5057A3, U28 DRV5057A3, U29 DRV5057A3, U3 DRV5057A3, U30 DRV5057A3, U31 DRV5057A3, U32 DRV5057A3, U33 DRV5057A3, U34 DRV5057A3, U4 DRV5057A3, U5 DRV5057A3, U6 DRV5057A3, U7 DRV5057A3, U8 DRV5057A3, U9 DRV5057A3

Commit message: finish left hand pcb
Parts:
- added LED1: LED_6028R, marbastlib-various:LED_6028R, symbol marbastlib-various:LED_6028R
- C1, C2, C3, C4, C5, C6: footprint (none) -> Capacitor_SMD:C_0402_1005Metric
- D1, D10, D11, D12, D13, D14, D15, D16, D17, D18, D19, D2, D20, D21, D22, D23, D24, D25, D26, D27, D28, D29, D3, D30, D31, D32, D4, D5, D6, D7, D8, D9: footprint (none) -> marbastlib-mx:LED_MX_6028R; symbol Device:LED_RGBA -> marbastlib-various:LED_6028R
- IC1: footprint QFN40P700X700X80-61N-D -> IS31FL3741A-QFLS4-TR:QFN40P700X700X80-61N-D
- J1: footprint (none) -> Connector_USB:USB_C_Receptacle_Amphenol_12401610E4-2A
- R1, R10, R11, R12, R13, R14, R15, R16, R17, R18, R2, R3, R4, R5, R6, R7, R8, R9: footprint (none) -> Resistor_SMD:R_0603_1608Metric
- U1, U10, U11, U12, U13, U14, U15, U16, U17, U18, U19, U2, U20, U21, U22, U23, U26, U27, U28, U29, U3, U30, U31, U32, U33, U34, U4, U5, U6, U7, U8, U9: footprint Package_TO_SOT_SMD:SOT-23 -> lib:DRV5057A3_K
Connections:
- net R_G_1: now also D10.1 (GK), D14.1 (GK), D19.1 (GK), D24.1 (GK), D28.1 (GK), D5.1 (GK); no longer D10.2 (GK), D14.2 (GK), D19.2 (GK), D24.2 (GK), D28.2 (GK), D5.2 (GK)
- net R_G_2: now also D11.1 (GK), D15.1 (GK), D20.1 (GK), D25.1 (GK), D29.1 (GK), D6.1 (GK); no longer D11.2 (GK), D15.2 (GK), D20.2 (GK), D25.2 (GK), D29.2 (GK), D6.2 (GK)
- net R_G_3: now also D12.1 (GK), D16.1 (GK), D21.1 (GK), D26.1 (GK), D30.1 (GK), D7.1 (GK); no longer D12.2 (GK), D16.2 (GK), D21.2 (GK), D26.2 (GK), D30.2 (GK), D7.2 (GK)
- net R_G_4: now also D1.1 (GK), D13.1 (GK), D17.1 (GK), D22.1 (GK), D27.1 (GK), D3.1 (GK), D31.1 (GK), D8.1 (GK); no longer D1.2 (GK), D13.2 (GK), D17.2 (GK), D22.2 (GK), D27.2 (GK), D3.2 (GK), D31.2 (GK), D8.2 (GK)
- net R_G_5: now also D18.1 (GK), D2.1 (GK), D23.1 (GK), D32.1 (GK), D4.1 (GK), D9.1 (GK); no longer D18.2 (GK), D2.2 (GK), D23.2 (GK), D32.2 (GK), D4.2 (GK), D9.2 (GK)
- net R_R_1: now also D10.2 (RK), D14.2 (RK), D19.2 (RK), D24.2 (RK), D28.2 (RK), D5.2 (RK); no longer D10.1 (RK), D14.1 (RK), D19.1 (RK), D24.1 (RK), D28.1 (RK), D5.1 (RK)
- net R_R_2: now also D11.2 (RK), D15.2 (RK), D20.2 (RK), D25.2 (RK), D29.2 (RK), D6.2 (RK); no longer D11.1 (RK), D15.1 (RK), D20.1 (RK), D25.1 (RK), D29.1 (RK), D6.1 (RK)
- net R_R_3: now also D12.2 (RK), D16.2 (RK), D21.2 (RK), D26.2 (RK), D30.2 (RK), D7.2 (RK); no longer D12.1 (RK), D16.1 (RK), D21.1 (RK), D26.1 (RK), D30.1 (RK), D7.1 (RK)
- net R_R_4: now also D1.2 (RK), D13.2 (RK), D17.2 (RK), D22.2 (RK), D27.2 (RK), D3.2 (RK), D31.2 (RK), D8.2 (RK); no longer D1.1 (RK), D13.1 (RK), D17.1 (RK), D22.1 (RK), D27.1 (RK), D3.1 (RK), D31.1 (RK), D8.1 (RK)
- net R_R_5: now also D18.2 (RK), D2.2 (RK), D23.2 (RK), D32.2 (RK), D4.2 (RK), D9.2 (RK); no longer D18.1 (RK), D2.1 (RK), D23.1 (RK), D32.1 (RK), D4.1 (RK), D9.1 (RK)
- net at U15.2 (OUT): now also U24.8 (I1); no longer U24.2 (I7)
- net at U6.2 (OUT): now also U24.21 (I10); no longer U24.20 (I11)
- net at U28.2 (OUT): now also U25.3 (I6); no longer U24.8 (I1)
- net at U20.2 (OUT): now also U25.19 (I12); no longer U25.22 (I9)
- net at U22.2 (OUT): now also U25.21 (I10); no longer U25.2 (I7)
- net at U34.2 (OUT): now also U25.9 (I0); no longer U25.20 (I11)
- net at U27.2 (OUT): now also U25.2 (I7); no longer U24.7 (I2)
- net at U8.2 (OUT): now also U24.23 (I8); no longer U24.22 (I9)
- net at U29.2 (OUT): now also U25.4 (I5); no longer U24.9 (I0)
- net at U19.2 (OUT): now also U25.18 (I13); no longer U25.21 (I10)
- net at U7.2 (OUT): now also U24.22 (I9); no longer U24.21 (I10)
- net at U5.2 (OUT): now also U24.20 (I11); no longer U25.9 (I0)
- net at U12.2 (OUT): now also U24.4 (I5); no longer U25.6 (I3)
- net at U26.2 (OUT): now also U25.23 (I8); no longer U24.6 (I3)
- net at U33.2 (OUT): now also U25.8 (I1); no longer U25.19 (I12)
- net at U21.2 (OUT): now also U25.20 (I11); no longer U25.23 (I8)
- net at U14.2 (OUT): now also U24.7 (I2); no longer U24.23 (I8)
- net at U17.2 (OUT): now also U25.16 (I15); no longer U24.4 (I5)
- net at U31.2 (OUT): now also U25.6 (I3); no longer U25.17 (I14)
- net at U30.2 (OUT): now also U25.5 (I4); no longer U25.16 (I15)
- net at U32.2 (OUT): now also U25.7 (I2); no longer U25.18 (I13)
- net at U23.2 (OUT): now also U25.22 (I9); no longer U25.3 (I6)
- net at U10.2 (OUT): now also U24.2 (I7); no longer U25.4 (I5)
- net at U11.2 (OUT): now also U24.3 (I6); no longer U25.5 (I4)
- net at U13.2 (OUT): now also U24.5 (I4); no longer U25.7 (I2)
- net at U9.2 (OUT): now also U24.6 (I3); no longer U25.8 (I1)
- net at U18.2 (OUT): now also U25.17 (I14); no longer U24.5 (I4)
- net at U16.2 (OUT): now also U24.9 (I0); no longer U24.3 (I6)
Other:
- moved on the sheet: U24, U25, U9

Commit message: whatever the fuck i all did
Parts:
- removed C1, C3, C5: 1uF, Capacitor_SMD:C_0402_1005Metric, symbol Device:C_Small
- removed C2, C4, C6: 0.1uF, Capacitor_SMD:C_0402_1005Metric, symbol Device:C_Small
- removed D1, D10, D11, D12, D13, D14, D15, D16, D17, D18, D19, D2, D20, D21, D22, D23, D24, D25, D26, D27, D28, D29, D3, D30, D31, D32, D4, D5, D6, D7, D8, D9: LED_RGB, marbastlib-mx:LED_MX_6028R, symbol marbastlib-various:LED_6028R
- removed IC1: IS31FL3741A-QFLS4-TR, IS31FL3741A-QFLS4-TR:QFN40P700X700X80-61N-D, symbol IS31FL3741A-QFLS4-TR:IS31FL3741A-QFLS4-TR
- removed LED1: LED_6028R, marbastlib-various:LED_6028R, symbol marbastlib-various:LED_6028R
- removed R1: 10k, Resistor_SMD:R_0603_1608Metric, symbol Device:R
- removed R10, R13, R16, R4, R7: 51, Resistor_SMD:R_0603_1608Metric, symbol Device:R
- removed R11, R12, R14, R15, R17, R18, R5, R6, R8, R9: 20, Resistor_SMD:R_0603_1608Metric, symbol Device:R
- removed R2, R3: 2k, Resistor_SMD:R_0603_1608Metric, symbol Device:R
- added C34, C38: 10uF, Capacitor_SMD:C_0603_1608Metric, symbol pspice:CAP
- added LED10, LED11, LED12, LED13, LED14, LED15, LED16, LED17, LED18, LED19, LED2, LED20, LED21, LED22, LED23, LED24, LED25, LED26, LED27, LED28, LED29, LED3, LED30, LED31, LED32, LED33, LED4, LED5, LED6, LED7, LED8, LED9: MX_SK6812MINI-E, lib:LED_MX_SK6812MINI-R, symbol marbastlib-mx:MX_SK6812MINI-E
- added U73: NCP1117-3.3_SOT223, Package_TO_SOT_SMD:SOT-223-3_TabPin2, symbol Regulator_Linear:NCP1117-3.3_SOT223
Connections:
- net +3.3V: now also C38.1, U73.2 (VO); no longer J1.A4 (VBUS), J1.A9 (VBUS), J1.B4 (VBUS), J1.B9 (VBUS)
- net GND: now also J1.B5 (CC2), C34.2, C38.2, LED10.4 (VSS), LED11.4 (VSS), LED12.4 (VSS), LED13.4 (VSS), LED14.4 (VSS), LED15.4 (VSS), LED16.4 (VSS), LED17.4 (VSS), LED18.4 (VSS), LED19.4 (VSS), LED2.4 (VSS), LED20.4 (VSS), LED21.4 (VSS), LED22.4 (VSS), LED23.4 (VSS), LED24.4 (VSS), LED25.4 (VSS), LED26.4 (VSS), LED28.4 (VSS), LED29.4 (VSS), LED3.4 (VSS), LED30.4 (VSS), LED4.4 (VSS), LED5.4 (VSS), LED6.4 (VSS), LED7.4 (VSS), LED8.4 (VSS), LED9.4 (VSS), U73.1 (GND)
- net MUX3 S0: no longer J1.A2 (TX1+)
- net MUX3 S1: no longer J1.A3 (TX1-)
- net MUX3 S2: no longer J1.B11 (RX1+)
- net MUX3 S3: no longer J1.B10 (RX1-)
- net MUX4 S0: no longer J1.B2 (TX2+)
- net MUX4 S1: no longer J1.B3 (TX2-)
- net MUX4 S2: no longer J1.A11 (RX2+)
- net MUX4 S3: no longer J1.A10 (RX2-)
- net +5V: now reaches J1.A5 (CC1)
- net +5V: now also J1.A4 (VBUS), J1.A9 (VBUS), J1.B4 (VBUS), J1.B9 (VBUS), C34.1, LED10.1 (VDD), LED11.1 (VDD), LED12.1 (VDD), LED13.1 (VDD), LED14.1 (VDD), LED15.1 (VDD), LED16.1 (VDD), LED17.1 (VDD), LED18.1 (VDD), LED19.1 (VDD), LED2.1 (VDD), LED20.1 (VDD), LED21.1 (VDD), LED22.1 (VDD), LED23.1 (VDD), LED24.1 (VDD), LED25.1 (VDD), LED26.1 (VDD), LED27.1 (VDD), LED28.1 (VDD), LED29.1 (VDD), LED3.1 (VDD), LED30.1 (VDD), LED31.1 (VDD), LED32.1 (VDD), LED33.1 (VDD), LED4.1 (VDD), LED5.1 (VDD), LED6.1 (VDD), LED7.1 (VDD), LED8.1 (VDD), LED9.1 (VDD), U73.3 (VI)
- net I2C SCL renamed LED_USB
- net LED_USB: now also LED2.3 (DIN)
- net I2C SDA: no longer names the net of J1.A6 (D+)
- net I2C SDA: no longer J1.B6 (D+)
- new net: LED2.2 (DOUT), LED3.3 (DIN)
- new net: LED8.2 (DOUT), LED9.3 (DIN)
- new net: LED7.2 (DOUT), LED8.3 (DIN)
- new net: LED23.2 (DOUT), LED24.3 (DIN)
- new net: LED22.2 (DOUT), LED23.3 (DIN)
- new net: LED18.2 (DOUT), LED19.3 (DIN)
- new net: LED17.2 (DOUT), LED18.3 (DIN)
- new net: LED10.3 (DIN), LED9.2 (DOUT)
- new net: LED29.2 (DOUT), LED30.3 (DIN)
- new net: LED28.2 (DOUT), LED29.3 (DIN)
- new net: LED19.2 (DOUT), LED20.3 (DIN)
- new net: LED15.2 (DOUT), LED16.3 (DIN)
- new net: LED14.2 (DOUT), LED15.3 (DIN)
- new net: LED26.2 (DOUT), LED28.3 (DIN)
- new net: LED25.2 (DOUT), LED26.3 (DIN)
- new net: LED24.2 (DOUT), LED25.3 (DIN)
- new net: LED27.2 (DOUT), LED31.3 (DIN)
- new net: LED27.3 (DIN), LED30.2 (DOUT)
- new net: LED27.4 (VSS), LED31.4 (VSS), LED32.4 (VSS), LED33.4 (VSS)
- new net: LED20.2 (DOUT), LED21.3 (DIN)
- new net: LED10.2 (DOUT), LED11.3 (DIN)
- new net: LED32.2 (DOUT), LED33.3 (DIN)
- new net: LED13.2 (DOUT), LED14.3 (DIN)
- new net: LED12.2 (DOUT), LED13.3 (DIN)
- new net: LED16.2 (DOUT), LED17.3 (DIN)
- new net: LED5.2 (DOUT), LED6.3 (DIN)
- new net: LED4.2 (DOUT), LED5.3 (DIN)
- new net: LED11.2 (DOUT), LED12.3 (DIN)
- new net: LED31.2 (DOUT), LED32.3 (DIN)
- new net: LED3.2 (DOUT), LED4.3 (DIN)
- new net: LED6.2 (DOUT), LED7.3 (DIN)
- new net: LED21.2 (DOUT), LED22.3 (DIN)
- new net MUX S0: J1.A2 (TX1+), J1.B2 (TX2+)
- new net MUX S1: J1.A3 (TX1-), J1.B3 (TX2-)
- new net MUX S2: J1.A11 (RX2+), J1.B11 (RX1+)
- new net MUX S3: J1.A10 (RX2-), J1.B10 (RX1-)

Commit message: redox woodox left hand pcb
Parts:
- added C1, C7, C9: 0.1uF, Capacitor_SMD:C_0603_1608Metric, symbol Device:C_Small
- added C10, C6: 10uF, Capacitor_SMD:C_0603_1608Metric, symbol pspice:CAP
- added C2, C3: 27pF, Capacitor_SMD:C_0603_1608Metric, symbol Device:C_Small
- added C4, C5, C8: 1uF, Capacitor_SMD:C_0603_1608Metric, symbol Device:C_Small
- added IC1: W25Q16JVUXIQ_TR, W25Q16JVUXIQ_TR:SON50P300X200X60-9N, symbol W25Q16JVUXIQ_TR:W25Q16JVUXIQ_TR
- added J2: Conn_01x03_Female, Connector_PinHeader_2.54mm:PinHeader_1x04_P2.54mm_Vertical, symbol Connector:Conn_01x04_Female
- added J3: USB_C_Receptacle, Connector_USB:USB_C_Receptacle_Amphenol_12401610E4-2A, symbol Connector:USB_C_Receptacle
- added R1, R3, R8: 1k, Resistor_SMD:R_0603_1608Metric, symbol Device:R
- added R2: 10k, Resistor_SMD:R_0603_1608Metric, symbol Device:R
- added R4, R5: 27.4, Resistor_SMD:R_0603_1608Metric, symbol Device:R
- added R6, R7: 5k1, Resistor_SMD:R_0603_1608Metric, symbol Device:R
- added SW1: BOOT, Button_Switch_SMD:SW_Push_1P1T_NO_Vertical_Wuerth_434133025816, symbol Switch:SW_Push
- added SW2: RESET, Button_Switch_SMD:SW_Push_1P1T_NO_Vertical_Wuerth_434133025816, symbol Switch:SW_Push
- added U16: NCP1117-3.3_SOT223, Package_TO_SOT_SMD:SOT-223-3_TabPin2, symbol Regulator_Linear:NCP1117-3.3_SOT223
- added U3: RP2040, Package_DFN_QFN:QFN-56-1EP_7x7mm_P0.4mm_EP3.2x3.2mm, symbol MCU_RaspberryPi:RP2040
- added Y1: ECS-120-8-30-JGN-TR, Crystal:Crystal_SMD_5032-2Pin_5.0x3.2mm, symbol Device:Crystal
- renumbered C34 to C11, C38 to C12, LED31 to LED1, LED9 to LED10, LED18 to LED11, LED21 to LED12, LED30 to LED13, LED5 to LED14, LED10 to LED15, LED17 to LED16, LED22 to LED17, LED29 to LED18, LED4 to LED19, LED32 to LED2, LED11 to LED20, LED16 to LED21, LED23 to LED22, LED28 to LED23, LED3 to LED24, LED12 to LED25, LED15 to LED26, LED24 to LED27, LED2 to LED28, LED13 to LED29, LED27 to LED3, LED14 to LED30, LED25 to LED31, LED26 to LED32, LED33 to LED4, LED7 to LED5, LED8 to LED6, LED19 to LED7, LED20 to LED8, LED6 to LED9, U24 to U10, U10 to U11, U11 to U12, U12 to U13, U13 to U14, U9 to U15, U14 to U17, U15 to U18, U16 to U19, U17 to U20, U18 to U21, U19 to U22, U20 to U23, U21 to U24, U22 to U25, U23 to U26, U26 to U27, U27 to U28, U28 to U29, U29 to U30, U25 to U31, U30 to U32, U31 to U33, U32 to U34, U33 to U35, U34 to U36, U73 to U37, U3 to U4, U4 to U5, U5 to U6, U6 to U7, U7 to U8, U8 to U9
Connections:
- net +3.3V: now also C10.1, C8.1, J2.1 (Pin_1), U16.2 (VO), U3.1 (IOVDD), U3.10 (IOVDD), U3.22 (IOVDD), U3.33 (IOVDD), U3.42 (IOVDD), U3.49 (IOVDD)
- net +5V: now also J3.A4 (VBUS), J3.A9 (VBUS), J3.B4 (VBUS), J3.B9 (VBUS), U16.3 (VI); no longer LED1.1 (VDD), LED10.1 (VDD), LED11.1 (VDD), LED12.1 (VDD), LED13.1 (VDD), LED14.1 (VDD), LED15.1 (VDD), LED16.1 (VDD), LED17.1 (VDD), LED18.1 (VDD), LED19.1 (VDD), LED2.1 (VDD), LED20.1 (VDD), LED21.1 (VDD), LED22.1 (VDD), LED23.1 (VDD), LED24.1 (VDD), LED25.1 (VDD), LED26.1 (VDD), LED27.1 (VDD), LED28.1 (VDD), LED29.1 (VDD), LED3.1 (VDD), LED30.1 (VDD), LED31.1 (VDD), LED32.1 (VDD), LED4.1 (VDD), LED5.1 (VDD), LED6.1 (VDD), LED7.1 (VDD), LED8.1 (VDD), LED9.1 (VDD)
- net GND: now also C1.2, C10.2, C4.2, C5.1, C6.2, C7.1, C8.2, C9.1, IC1.4 (GND), IC1.9 (EP), J2.4 (Pin_4), J3.A1 (GND), J3.A12 (GND), J3.B1 (GND), J3.B12 (GND), SW1.1, SW2.1, U16.1 (GND), U3.19 (TESTEN), U3.57 (GND); no longer LED11.4 (VSS), LED12.4 (VSS), LED13.4 (VSS), LED16.4 (VSS), LED17.4 (VSS), LED18.4 (VSS), LED21.4 (VSS), LED22.4 (VSS), LED23.4 (VSS), LED26.4 (VSS), LED27.4 (VSS), LED30.4 (VSS), LED31.4 (VSS), LED32.4 (VSS), LED7.4 (VSS), LED8.4 (VSS)
- new net: R8.1, SW2.2
- new net: R8.2, U3.26 (RUN)
- new net: IC1.8 (VCC), R2.2
- new net: C3.1, Y1.2
- new net: LED10.1 (VDD), LED11.1 (VDD), LED15.1 (VDD), LED16.1 (VDD), LED20.1 (VDD), LED21.1 (VDD), LED25.1 (VDD), LED26.1 (VDD), LED29.1 (VDD), LED30.1 (VDD), LED6.1 (VDD), LED7.1 (VDD)
- new net: R1.1, SW1.2
- new net: LED12.1 (VDD), LED13.1 (VDD), LED17.1 (VDD), LED18.1 (VDD), LED22.1 (VDD), LED23.1 (VDD), LED31.1 (VDD), LED32.1 (VDD), LED4.1 (VDD)
- new net: LED11.4 (VSS), LED12.4 (VSS), LED16.4 (VSS), LED17.4 (VSS), LED21.4 (VSS), LED22.4 (VSS), LED26.4 (VSS), LED27.4 (VSS), LED30.4 (VSS), LED31.4 (VSS), LED7.4 (VSS), LED8.4 (VSS)
- new net: C2.1, Y1.1
- new net: J3.B5 (CC2), R6.1
- new net: R6.2, R7.2
- new net: J3.A5 (CC1), R7.1
- new net: C2.2, R3.1
- new net: R3.2, U3.21 (XOUT)
- new net: C5.2, U3.23 (DVDD), U3.50 (DVDD)
- new net: J2.3 (Pin_3), U3.24 (SWCLK)
- new net: J2.2 (Pin_2), U3.25 (SWD)
- new net: C9.2, U3.45 (VREG_VOUT)
- new net: R4.2, U3.46 (USB_DM)
- new net: R5.2, U3.47 (USB_DP)
- new net: J3.B6 (D+), R5.1
- new net: J3.A7 (D-), J3.B7 (D-)
- new net LED: U3.7 (GPIO5)
- new net MUX1 COM: U3.38 (GPIO26_ADC0)
- new net MUX1 S0: U3.6 (GPIO4)
- new net MUX1 S1: U3.5 (GPIO3)
- new net MUX1 S2: U3.4 (GPIO2)
- new net MUX1 S3: U3.3 (GPIO1)
- new net QSPI_SCLK: IC1.6 (CLK), U3.52 (QSPI_SCLK)
- new net QSPI_SD0: IC1.5 (DI(IO0)), U3.53 (QSPI_SD0)
- new net QSPI_SD1: IC1.2 (DO(IO1)), U3.55 (QSPI_SD1)
- new net QSPI_SD2: IC1.3 (IO2), U3.54 (QSPI_SD2)
- new net QSPI_SD3: IC1.7 (IO3), U3.51 (QSPI_SD3)
- new net QSPI_SS: IC1.1 (~{CS}), R1.2, R2.1, U3.56 (QSPI_SS)
Other:
- moved on the sheet: C11, C12, J1, LED1, LED10, LED11, LED12, LED13, LED14, LED15, LED16, LED17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
