File: woodox/woodox.kicad_pcb (KiCad board)
At the start: 4 copper layers, 162.2 x 126.5 mm, 224 parts, among them J1 Conn_01x03_Female, J2 USB_C_To_Host, J4 USB_C_To_Host, J5 Conn_01x05_Socket, J6 USB_C_Interlink, J7 USB_C_Interlink, J8 Conn_01x05_Socket, SW1 SW_Push, SW2 SW_Push, SW3 SW_Push, SW4 SW_Push, U1 DRV5057A3, U10 OLED_256x64_I2C, U11 DRV5057A3, U12 DRV5057A3, U13 DRV5057A3, U14 DRV5057A3, U15 DRV5057A3, U16 DRV5057A3, U17 DRV5057A3, U18 DRV5057A3, U19 DRV5057A3, U2 DRV5057A3, U20 DRV5057A3, U21 DRV5057A3, U22 DRV5057A3, U23 DRV5057A3, U24 DRV5057A3, U25 W25Q128JVP, U26 DRV5057A3, U27 DRV5057A3, U28 DRV5057A3, U29 DRV5057A3, U3 DRV5057A3, U30 DRV5057A3, U31 DRV5057A3, U32 DRV5057A3, U33 NCP1117-3.3_SOT223, U34 74HC4051, U35 74HC4051, U36 74HC4051, U37 74HC4051, U38 DRV5057A3, U39 DRV5057A3, U4 DRV5057A3, U40 DRV5057A3, U41 DRV5057A3, U42 DRV5057A3, U43 DRV5057A3, U44 DRV5057A3, U45 DRV5057A3, U46 DRV5057A3, U47 DRV5057A3, U48 DRV5057A3, U49 W25Q128JVP, U5 DRV5057A3, U50 DRV5057A3, U51 DRV5057A3, U52 DRV5057A3, U53 DRV5057A3, U54 DRV5057A3, U55 DRV5057A3, U56 DRV5057A3, U57 DRV5057A3, U58 DRV5057A3, U59 DRV5057A3, U6 DRV5057A3, U60 DRV5057A3, U61 DRV5057A3, U62 DRV5057A3, U63 DRV5057A3, U64 RP2350_80QFN, U65 DRV5057A3, U66 DRV5057A3, U67 DRV5057A3, U68 DRV5057A3, U69 DRV5057A3, U7 DRV5057A3, U70 DRV5057A3, U71 DRV5057A3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

Commit message: fix lints
Parts:
- U64, U79: footprint Package_DFN_QFN:QFN-80-1EP_10x10mm_P0.4mm_EP3.4x3.4mm_ThermalVias -> RP2350_80QFN_minimal:RP2350-QFN-80-1EP_10x10_P0.4mm_EP3.4x3.4mm_ThermalVias
- moved J1 0.92 mm to (152.7, 33.0)
- moved C37 0.50 mm to (160.0, 84.5)
- moved C50 0.50 mm to (161.0, 84.5)
- moved C26 0.20 mm to (160.9, 67.3)
- moved C18 0.19 mm to (159.9, 67.4)
Routing:
- net Net-(U28-OUT): track 2.22 -> 13.8 mm, vias 0 -> 2
- net Net-(U26-OUT): track 30.4 -> 19.9 mm
- net GND: track 16.9 -> 25.0 mm, vias 47 -> 75
- net +3.3VR: track 1140.1 -> 1133.6 mm
- net +1V1: track 58.7 -> 62.8 mm
- net /MUX R E: track 117.4 -> 114.0 mm, vias 7 -> 6
- net /MUX1 COM: track 57.3 -> 54.6 mm, vias 1 -> 2
- net Net-(U30-OUT): track 19.6 -> 17.1 mm
- net /D_CS_R: track 44.6 -> 42.3 mm
- net +5V: track 1499.5 -> 1498.2 mm, vias 83 -> 81
- net /MUX R S0: track 105.5 -> 104.6 mm, vias 5 -> 4
- net +3.3V: track 1053.6 -> 1054.2 mm
- net /D_CS: track 29.6 -> 29.0 mm
- net /QSPI_R_SD1: track 14.2 -> 13.7 mm
- net /QSPI_R_SD2: track 12.7 -> 12.2 mm
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