File: woodox/woodox.kicad_pcb (KiCad board)
At the start: 4 copper layers, 162.2 x 126.5 mm, 233 parts, among them J1 Conn_01x03_Female, J10 Conn_01x01, J11 Conn_01x01, J12 Conn_01x01, J2 USB_C_To_Host, J3 Conn_01x03_Female, J4 USB_C_To_Host, J5 Conn_01x05_Socket, J6 USB_C_Interlink, J7 USB_C_Interlink, J8 Conn_01x05_Socket, J9 Conn_01x01, SW1 SW_Push, SW2 SW_Push, SW3 SW_Push, SW4 SW_Push, U1 DRV5057A3, U10 OLED_256x64_I2C, U11 DRV5057A3, U12 DRV5057A3, U13 DRV5057A3, U14 DRV5057A3, U15 DRV5057A3, U16 DRV5057A3, U17 DRV5057A3, U18 DRV5057A3, U19 DRV5057A3, U2 DRV5057A3, U20 DRV5057A3, U21 DRV5057A3, U22 DRV5057A3, U23 DRV5057A3, U24 DRV5057A3, U25 W25Q128JVP, U26 DRV5057A3, U27 DRV5057A3, U28 DRV5057A3, U29 DRV5057A3, U3 DRV5057A3, U30 DRV5057A3, U31 DRV5057A3, U32 DRV5057A3, U33 NCP1117-3.3_SOT223, U34 74HC4051, U35 74HC4051, U36 74HC4051, U37 74HC4051, U38 DRV5057A3, U39 DRV5057A3, U4 DRV5057A3, U40 DRV5057A3, U41 DRV5057A3, U42 DRV5057A3, U43 DRV5057A3, U44 DRV5057A3, U45 DRV5057A3, U46 DRV5057A3, U47 DRV5057A3, U48 DRV5057A3, U49 W25Q128JVP, U5 DRV5057A3, U50 DRV5057A3, U51 DRV5057A3, U52 DRV5057A3, U53 DRV5057A3, U54 DRV5057A3, U55 DRV5057A3, U56 DRV5057A3, U57 DRV5057A3, U58 DRV5057A3, U59 DRV5057A3, U6 DRV5057A3, U60 DRV5057A3, U61 DRV5057A3, U62 DRV5057A3, U63 DRV5057A3, U64 RP2350_80QFN, U65 DRV5057A3, U66 DRV5057A3, U67 DRV5057A3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

Commit message: idk
Parts:
- C10, C16, C20, C6: footprint Capacitor_SMD:C_0603_1608Metric -> Capacitor_SMD:C_0402_1005Metric
- R1, R11, R13, R14, R15, R16, R17, R18, R19, R2, R20, R23, R6, R7: footprint Resistor_SMD:R_0603_1608Metric -> Resistor_SMD:R_0402_1005Metric
Connections:
- U25 pad 9: GND -> (no net)
- U49 pad 9: GND -> (no net)
Routing:
- net +5V: track 1501.8 -> 1502.6 mm
- net /QSPI_SS: track 38.2 -> 38.8 mm
- net /QSPI_R_SS: track 33.6 -> 34.2 mm
- net Net-(J4-CC1): track 12.5 -> 13.2 mm
- net +3.3V: track 1081.0 -> 1081.6 mm
- net +1V1: track 62.8 -> 63.3 mm
