File: woodox/woodox.kicad_sch (KiCad schematic)
At the start: 0 parts

Commit message: redox woodox left hand pcb
Parts:
- added C1, C7, C9: 0.1uF, Capacitor_SMD:C_0603_1608Metric, symbol Device:C_Small
- added C10, C6: 10uF, Capacitor_SMD:C_0603_1608Metric, symbol pspice:CAP
- added C2, C3: 27pF, Capacitor_SMD:C_0603_1608Metric, symbol Device:C_Small
- added C4, C5, C8: 1uF, Capacitor_SMD:C_0603_1608Metric, symbol Device:C_Small
- added IC1: W25Q16JVUXIQ_TR, W25Q16JVUXIQ_TR:SON50P300X200X60-9N, symbol W25Q16JVUXIQ_TR:W25Q16JVUXIQ_TR
- added J1: Conn_01x03_Female, Connector_PinHeader_2.54mm:PinHeader_1x04_P2.54mm_Vertical, symbol Connector:Conn_01x04_Female
- added J2: USB_C_Receptacle, Connector_USB:USB_C_Receptacle_Amphenol_12401610E4-2A, symbol Connector:USB_C_Receptacle
- added LED1, LED10, LED11, LED12, LED13, LED14, LED15, LED16, LED17, LED18, LED19, LED2, LED20, LED21, LED22, LED23, LED24, LED25, LED26, LED27, LED28, LED29, LED3, LED30, LED31, LED32, LED4, LED5, LED6, LED7, LED8, LED9: MX_SK6812MINI-E, lib:LED_MX_SK6812MINI-R, symbol marbastlib-mx:MX_SK6812MINI-E
- added R1, R3, R8: 1k, Resistor_SMD:R_0603_1608Metric, symbol Device:R
- added R2: 10k, Resistor_SMD:R_0603_1608Metric, symbol Device:R
- added R4, R5: 27.4, Resistor_SMD:R_0603_1608Metric, symbol Device:R
- added R6, R7: 5k1, Resistor_SMD:R_0603_1608Metric, symbol Device:R
- added SW1: BOOT, Button_Switch_SMD:SW_Push_1P1T_NO_Vertical_Wuerth_434133025816, symbol Switch:SW_Push
- added SW2: RESET, Button_Switch_SMD:SW_Push_1P1T_NO_Vertical_Wuerth_434133025816, symbol Switch:SW_Push
- added U1, U11, U12, U13, U14, U15, U16, U17, U18, U19, U2, U20, U21, U22, U23, U24, U26, U27, U28, U29, U3, U30, U31, U32, U38, U39, U4, U5, U6, U7, U8, U9: DRV5057A3, lib:DRV5057A3_K, symbol Sensor_Magnetic:DRV5055A3xDBZxQ1
- added U10: OLED_256x64_I2C, Connector_PinHeader_2.54mm:PinHeader_1x07_P2.54mm_Vertical, symbol oled_256x64_i2c:OLED_256x64_I2C
- added U25: RP2040, Package_DFN_QFN:QFN-56-1EP_7x7mm_P0.4mm_EP3.2x3.2mm, symbol MCU_RaspberryPi:RP2040
- added U33: NCP1117-3.3_SOT223, Package_TO_SOT_SMD:SOT-223-3_TabPin2, symbol Regulator_Linear:NCP1117-3.3_SOT223
- added U34, U35, U36, U37: 74HC4051, Package_SO:TSSOP-16_4.4x5mm_P0.65mm, symbol 74xx:74HC4051
- added Y1: ECS-120-8-30-JGN-TR, Crystal:Crystal_SMD_5032-2Pin_5.0x3.2mm, symbol Device:Crystal
Connections:
- new net: LED24.2 (DOUT), LED29.3 (DIN)
- new net: LED19.2 (DOUT), LED24.3 (DIN)
- new net: LED18.3 (DIN), LED23.2 (DOUT)
- new net: LED23.3 (DIN), LED28.2 (DOUT)
- new net: LED20.2 (DOUT), LED25.3 (DIN)
- new net: LED15.2 (DOUT), LED20.3 (DIN)
- new net: U34.15 (A2), U5.2 (OUT)
- new net: U37.13 (A0), U9.2 (OUT)
- new net: LED29.2 (DOUT), LED31.3 (DIN)
- new net: U28.2 (OUT), U35.1 (A4)
- new net: U35.12 (A3), U38.2 (OUT)
- new net: U35.13 (A0), U7.2 (OUT)
- new net: U2.2 (OUT), U35.14 (A1)
- new net: U15.2 (OUT), U35.15 (A2)
- new net: U22.2 (OUT), U35.2 (A6)
- new net: U17.2 (OUT), U35.4 (A7)
- new net: U12.2 (OUT), U35.5 (A5)
- new net: R8.1, SW2.2
- new net: U16.2 (OUT), U34.4 (A7)
- new net: LED12.3 (DIN), LED8.2 (DOUT)
- new net: LED3.2 (DOUT), LED8.3 (DIN)
- new net: LED2.3 (DIN), LED7.2 (DOUT)
- new net: LED11.2 (DOUT), LED7.3 (DIN)
- new net: J2.A6 (D+), J2.B6 (D+), R5.1
- new net: R5.2, U25.47 (USB_DP)
- new net: U32.2 (OUT), U37.12 (A3)
- new net: LED21.3 (DIN), LED26.2 (DOUT)
- new net: LED25.2 (DOUT), LED26.3 (DIN)
- new net: C4.2, C7.2, C9.2, U25.23 (DVDD), U25.45 (VREG_VOUT), U25.50 (DVDD)
- new net: LED2.2 (DOUT), LED3.3 (DIN)
- new net: C2.1, Y1.1
- new net: C2.2, R3.1
- new net: U37.14 (A1), U4.2 (OUT)
- new net: C3.1, Y1.2
- new net: U3.2 (OUT), U36.14 (A1)
- new net: LED27.2 (DOUT), LED28.3 (DIN)
- new net: LED17.2 (DOUT), LED22.3 (DIN)
- new net: LED12.2 (DOUT), LED17.3 (DIN)
- new net: U30.2 (OUT), U37.1 (A4)
- new net: LED14.3 (DIN), LED5.2 (DOUT)
- new net: LED4.2 (DOUT), LED5.3 (DIN)
- new net: U13.2 (OUT), U36.5 (A5)
- new net: LED10.2 (DOUT), LED15.3 (DIN)
- new net: U23.2 (OUT), U36.2 (A6)
- new net: R1.1, SW1.2
- new net: LED13.2 (DOUT), LED9.3 (DIN)
- new net: LED13.3 (DIN), LED18.2 (DOUT)
- new net: LED4.3 (DIN), LED9.2 (DOUT)
- new net: C3.2, U25.20 (XIN)
- new net: LED11.3 (DIN), LED16.2 (DOUT)
- new net: LED14.2 (DOUT), LED19.3 (DIN)
- new net: U29.2 (OUT), U36.1 (A4)
- new net: U36.12 (A3), U39.2 (OUT)
- new net: U36.13 (A0), U8.2 (OUT)
- new net: U20.2 (OUT), U36.15 (A2)
- new net: U18.2 (OUT), U36.4 (A7)
- new net: J2.A5 (CC1), R7.1
- new net: J2.A7 (D-), J2.B7 (D-), R4.1
- new net: J2.B5 (CC2), R6.1
- new net: U11.2 (OUT), U34.5 (A5)
- new net: LED30.3 (DIN), LED32.2 (DOUT)
- new net: U24.2 (OUT), U37.2 (A6)
- new net: LED31.2 (DOUT), LED32.3 (DIN)
- new net: LED10.3 (DIN), LED6.2 (DOUT)
- new net: LED1.2 (DOUT), LED6.3 (DIN)
- new net: U19.2 (OUT), U37.4 (A7)
- new net: LED16.3 (DIN), LED21.2 (DOUT)
- new net: U26.2 (OUT), U37.15 (A2)
- new net: R3.2, U25.21 (XOUT)
- new net: LED22.2 (DOUT), LED27.3 (DIN)
- new net: U27.2 (OUT), U34.1 (A4)
- new net: U31.2 (OUT), U34.12 (A3)
- new net: U34.13 (A0), U6.2 (OUT)
- new net: U1.2 (OUT), U34.14 (A1)
- new net: U21.2 (OUT), U34.2 (A6)
- new net: U14.2 (OUT), U37.5 (A5)
- new net: J1.2 (Pin_2), U25.25 (SWD)
- new net: J1.3 (Pin_3), U25.24 (SWCLK)
- new net: R8.2, U25.26 (RUN)
- new net: R4.2, U25.46 (USB_DM)
- new net +3.3V: C1.1, C10.1, C5.1, C8.1, IC1.8 (VCC), J1.1 (Pin_1), R2.2, U1.1 (VCC), U10.2 (VCC), U11.1 (VCC), U12.1 (VCC), U13.1 (VCC), U14.1 (VCC), U15.1 (VCC), U16.1 (VCC), U17.1 (VCC), U18.1 (VCC), U19.1 (VCC), U2.1 (VCC), U20.1 (VCC), U21.1 (VCC), U22.1 (VCC), U23.1 (VCC), U24.1 (VCC), U25.1 (IOVDD), U25.10 (IOVDD), U25.22 (IOVDD), U25.33 (IOVDD), U25.42 (IOVDD), U25.43 (ADC_AVDD), U25.44 (VREG_IN), U25.48 (USB_VDD), U25.49 (IOVDD), U26.1 (VCC), U27.1 (VCC), U28.1 (VCC), U29.1 (VCC), U3.1 (VCC), U30.1 (VCC), U31.1 (VCC), U32.1 (VCC), U33.2 (VO), U34.16 (VCC), U35.16 (VCC), U36.16 (VCC), U37.16 (VCC), U38.1 (VCC), U39.1 (VCC), U4.1 (VCC), U5.1 (VCC), U6.1 (VCC), U7.1 (VCC), U8.1 (VCC), U9.1 (VCC)
- new net +5V: C6.1, J2.A4 (VBUS), J2.A9 (VBUS), J2.B4 (VBUS), J2.B9 (VBUS), LED1.1 (VDD), LED10.1 (VDD), LED11.1 (VDD), LED12.1 (VDD), LED13.1 (VDD), LED14.1 (VDD), LED15.1 (VDD), LED16.1 (VDD), LED17.1 (VDD), LED18.1 (VDD), LED19.1 (VDD), LED2.1 (VDD), LED20.1 (VDD), LED21.1 (VDD), LED22.1 (VDD), LED23.1 (VDD), LED24.1 (VDD), LED25.1 (VDD), LED26.1 (VDD), LED27.1 (VDD), LED28.1 (VDD), LED29.1 (VDD), LED3.1 (VDD), LED30.1 (VDD), LED31.1 (VDD), LED32.1 (VDD), LED4.1 (VDD), LED5.1 (VDD), LED6.1 (VDD), LED7.1 (VDD), LED8.1 (VDD), LED9.1 (VDD), U33.3 (VI)
- new net D_CS: U10.7 (CS), U25.13 (GPIO10)
- new net D_DC: U10.6 (DC), U25.12 (GPIO9)
- new net D_RST: U10.5 (RST), U25.11 (GPIO8)
- new net D_SCL: U10.3 (SCL), U25.8 (GPIO6)
- new net D_SDA: U10.4 (SDA), U25.9 (GPIO7)
- new net GND: C1.2, C10.2, C4.1, C5.2, C6.2, C7.1, C8.2, C9.1, IC1.4 (GND), IC1.9 (EP), J1.4 (Pin_4), J2.A1 (GND), J2.A12 (GND), J2.B1 (GND), J2.B12 (GND), LED1.4 (VSS), LED10.4 (VSS), LED11.4 (VSS), LED12.4 (VSS), LED13.4 (VSS), LED14.4 (VSS), LED15.4 (VSS), LED16.4 (VSS), LED17.4 (VSS), LED18.4 (VSS), LED19.4 (VSS), LED2.4 (VSS), LED20.4 (VSS), LED21.4 (VSS), LED22.4 (VSS), LED23.4 (VSS), LED24.4 (VSS), LED25.4 (VSS), LED26.4 (VSS), LED27.4 (VSS), LED28.4 (VSS), LED29.4 (VSS), LED3.4 (VSS), LED30.4 (VSS), LED31.4 (VSS), LED32.4 (VSS), LED4.4 (VSS), LED5.4 (VSS), LED6.4 (VSS), LED7.4 (VSS), LED8.4 (VSS), LED9.4 (VSS), R6.2, R7.2, SW1.1, SW2.1, U1.3 (GND), U10.1 (GND), U11.3 (GND), U12.3 (GND), U13.3 (GND), U14.3 (GND), U15.3 (GND), U16.3 (GND), U17.3 (GND), U18.3 (GND), U19.3 (GND), U2.3 (GND), U20.3 (GND), U21.3 (GND), U22.3 (GND), U23.3 (GND), U24.3 (GND), U25.19 (TESTEN), U25.57 (GND), U26.3 (GND), U27.3 (GND), U28.3 (GND), U29.3 (GND), U3.3 (GND), U30.3 (GND), U31.3 (GND), U32.3 (GND), U33.1 (GND), U34.7 (VEE), U34.8 (GND), U35.7 (VEE), U35.8 (GND), U36.7 (VEE), U36.8 (GND), U37.7 (VEE), U37.8 (GND), U38.3 (GND), U39.3 (GND), U4.3 (GND), U5.3 (GND), U6.3 (GND), U7.3 (GND), U8.3 (GND), U9.3 (GND)
- new net LED: LED1.3 (DIN), U25.32 (GPIO21)
- new net MUX E: U25.37 (GPIO25), U34.6 (~{E}), U35.6 (~{E}), U36.6 (~{E}), U37.6 (~{E})
- new net MUX S0: U25.36 (GPIO24), U34.11 (S0), U35.11 (S0), U36.11 (S0), U37.11 (S0)
- new net MUX S1: U25.35 (GPIO23), U34.10 (S1), U35.10 (S1), U36.10 (S1), U37.10 (S1)
- new net MUX S2: U25.34 (GPIO22), U34.9 (S2), U35.9 (S2), U36.9 (S2), U37.9 (S2)
- new net MUX1 COM: U25.41 (GPIO29_ADC3), U34.3 (A)
- new net MUX2 COM: U25.40 (GPIO28_ADC2), U35.3 (A)
- new net MUX3 COM: U25.39 (GPIO27_ADC1), U36.3 (A)
- new net MUX4 COM: U25.38 (GPIO26_ADC0), U37.3 (A)
- new net QSPI_SCLK: IC1.6 (CLK), U25.52 (QSPI_SCLK)
- new net QSPI_SD0: IC1.5 (DI(IO0)), U25.53 (QSPI_SD0)
- new net QSPI_SD1: IC1.2 (DO(IO1)), U25.55 (QSPI_SD1)
- new net QSPI_SD2: IC1.3 (IO2), U25.54 (QSPI_SD2)
- new net QSPI_SD3: IC1.7 (IO3), U25.51 (QSPI_SD3)
- new net QSPI_SS: IC1.1 (~{CS}), R1.2, R2.1, U25.56 (QSPI_SS)
Other:
- removed sheet Left Hand
- removed sheet Right Hand

Commit message: cleanup pcb
Parts:
- U1, U11, U12, U13, U14, U15, U16, U17, U18, U19, U2, U20, U21, U22, U23, U24, U26, U27, U28, U29, U3, U30, U31, U32, U38, U39, U4, U5, U6, U7, U8, U9: footprint lib:DRV5057A3_K -> lib:DRV505x
- U10: footprint Connector_PinHeader_2.54mm:PinHeader_1x07_P2.54mm_Vertical -> lib:OLED_256x64_I2C
Connections:
- net D_CS: now also U25.8 (GPIO6); no longer U25.13 (GPIO10)
- net D_DC: now also U25.9 (GPIO7); no longer U25.12 (GPIO9)
- net D_SCL: now also U25.13 (GPIO10); no longer U25.8 (GPIO6)
- net D_SDA: now also U25.12 (GPIO9); no longer U25.9 (GPIO7)
Changed lines of the file:
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@@
 	)
 	(label "D_SCL"
-		(at 256.54 157.48 270)
+		(at 246.38 157.48 270)
 		(effects
 			(font
@@
 	)
 	(label "D_SDA"
-		(at 254 157.48 270)
+		(at 248.92 157.48 270)
 		(effects
 			(font
@@
 	)
 	(label "D_DC"
-		(at 248.92 157.48 270)
+		(at 254 157.48 270)
 		(effects
 			(font
@@
 	)
 	(label "D_CS"
-		(at 246.38 157.48 270)
+		(at 256.54 157.48 270)
 		(effects
 			(font
@@
 			)
 		)
-		(property "Footprint" "lib:DRV5057A3_K"
+		(property "Footprint" "lib:DRV505x"
 			(at 123.19 328.93 0)
 			(effects
@@
 			)
 		)
-		(property "Footprint" "lib:DRV5057A3_K"
+		(property "Footprint" "lib:DRV505x"
 			(at 148.59 297.18 0)
 			(effects
@@
 			)
 		)
-		(property "Footprint" "lib:DRV5057A3_K"
+		(property "Footprint" "lib:DRV505x"
 			(at 199.39 217.17 0)
 			(effects
@@
 			)
 		)
-		(property "Footprint" "lib:DRV5057A3_K"
+		(property "Footprint" "lib:DRV505x"
 			(at 173.99 328.93 0)
 			(effects
@@
 			)
 		)
-		(property "Footprint" "lib:DRV5057A3_K"
+		(property "Footprint" "lib:DRV505x"
 			(at 288.29 337.82 0)
 			(effects
@@
 			)
 		)
-		(property "Footprint" "lib:DRV5057A3_K"
+		(property "Footprint" "lib:DRV505x"
 			(at 123.19 297.18 0)
 			(effects
@@
 			)
 		)
-		(property "Footprint" "lib:DRV5057A3_K"
+		(property "Footprint" "lib:DRV505x"
 			(at 123.19 270.51 0)
 			(effects
@@
 			)
 		)
-		(property "Footprint" "lib:DRV5057A3_K"
+		(property "Footprint" "lib:DRV505x"
 			(at 250.19 297.18 0)
 			(effects
@@
 			)
 		)
-		(property "Footprint" "lib:DRV5057A3_K"
+		(property "Footprint" "lib:DRV505x"
 			(at 173.99 270.51 0)
 			(effects
@@
 			)
 		)
-		(property "Footprint" "lib:DRV5057A3_K"
+		(property "Footprint" "lib:DRV505x"
 			(at 224.79 270.51 0)
 			(effects
@@
 			)
 		)
-		(property "Footprint" "lib:DRV5057A3_K"
+		(property "Footprint" "lib:DRV505x"
 			(at 123.19 243.84 0)
 			(effects
@@
 			)
 		)
-		(property "Footprint" "lib:DRV5057A3_K"
+		(property "Footprint" "lib:DRV505x"
 			(at 199.39 243.84 0)
 			(effects
@@
 			)
 		)
-		(property "Footprint" "lib:DRV5057A3_K"
+		(property "Footprint" "lib:DRV505x"
 			(at 309.88 337.82 0)
 			(effects
@@
 			)
 		)
-		(property "Footprint" "lib:DRV5057A3_K"
+		(property "Footprint" "lib:DRV505x"
 			(at 173.99 217.17 0)
 			(effects
@@
 			)
 		)
-		(property "Footprint" "lib:DRV5057A3_K"
+		(property "Footprint" "lib:DRV505x"
 			(at 173.99 243.84 0)
 			(effects
@@
 			)
 		)
-		(property "Footprint" "lib:DRV5057A3_K"
+		(property "Footprint" "lib:DRV505x"
 			(at 224.79 297.18 0)
 			(effects
@@
 			)
 		)
-		(property "Footprint" "lib:DRV5057A3_K"
+		(property "Footprint" "lib:DRV505x"
 			(at 199.39 297.18 0)
 			(effects
@@
 			)
 		)
-		(property "Footprint" "lib:DRV5057A3_K"
+		(property "Footprint" "lib:DRV505x"
 			(at 238.76 328.93 0)
 			(effects
@@
 			)
 		)
-		(property "Footprint" "lib:DRV5057A3_K"
+		(property "Footprint" "lib:DRV505x"
 			(at 199.39 270.51 0)
 			(effects
@@
 			)
 		)
-		(property "Footprint" "lib:DRV5057A3_K"
+		(property "Footprint" "lib:DRV505x"
 			(at 173.99 297.18 0)
 			(effects
@@
 			)
 		)
-		(property "Footprint" "lib:DRV5057A3_K"
+		(property "Footprint" "lib:DRV505x"
 			(at 250.19 270.51 0)
 			(effects
@@
 			)
 		)
-		(property "Footprint" "lib:DRV5057A3_K"
+		(property "Footprint" "lib:DRV505x"
 			(at 123.19 217.17 0)
 			(effects
@@
 			)
 		)
-		(property "Footprint" "lib:DRV5057A3_K"
+		(property "Footprint" "lib:DRV505x"
 			(at 199.39 328.93 0)
 			(effects
@@
 			)
 		)
-		(property "Footprint" "lib:DRV5057A3_K"
+		(property "Footprint" "lib:DRV505x"
 			(at 250.19 217.17 0)
 			(effects
@@
 			)
 		)
-		(property "Footprint" "Connector_PinHeader_2.54mm:PinHeader_1x07_P2.54mm_Vertical"
+		(property "Footprint" "lib:OLED_256x64_I2C"
 			(at 162.56 53.34 0)
 			(effects
@@
 			)
 		)
-		(property "Footprint" "lib:DRV5057A3_K"
+		(property "Footprint" "lib:DRV505x"
 			(at 309.88 312.42 0)
 			(effects
@@
 			)
 		)
-		(property "Footprint" "lib:DRV5057A3_K"
+		(property "Footprint" "lib:DRV505x"
 			(at 288.29 312.42 0)
 			(effects
@@
 			)
 		)
-		(property "Footprint" "lib:DRV5057A3_K"
+		(property "Footprint" "lib:DRV505x"
 			(at 148.59 243.84 0)
 			(effects
@@
 			)
 		)
-		(property "Footprint" "lib:DRV5057A3_K"
+		(property "Footprint" "lib:DRV505x"
 			(at 148.59 217.17 0)
 			(effects
@@
 			)
 		)
-		(property "Footprint" "lib:DRV5057A3_K"
+		(property "Footprint" "lib:DRV505x"
 			(at 250.19 243.84 0)
 			(effects
@@
 			)
 		)
-		(property "Footprint" "lib:DRV5057A3_K"
+		(property "Footprint" "lib:DRV505x"
 			(at 224.79 217.17 0)
 			(effects
@@
 			)
 		)
-		(property "Footprint" "lib:DRV5057A3_K"
+		(property "Footprint" "lib:DRV505x"
 			(at 148.59 270.51 0)
 			(effects
@@
 			)
 		)
-		(property "Footprint" "lib:DRV5057A3_K"
+		(property "Footprint" "lib:DRV505x"
 			(at 224.79 243.84 0)
 			(effects

Commit message: double sided pcb
Parts:
- added C11, C17, C19: 0.1uF, Capacitor_SMD:C_0603_1608Metric, symbol Device:C_Small
- added C12, C13: 27pF, Capacitor_SMD:C_0603_1608Metric, symbol Device:C_Small
- added C14, C15, C18: 1uF, Capacitor_SMD:C_0603_1608Metric, symbol Device:C_Small
- added C16, C20: 10uF, Capacitor_SMD:C_0603_1608Metric, symbol pspice:CAP
- added IC2: W25Q16JVUXIQ_TR, W25Q16JVUXIQ_TR:SON50P300X200X60-9N, symbol W25Q16JVUXIQ_TR:W25Q16JVUXIQ_TR
- added J4: USB_C_Receptacle, Connector_USB:USB_C_Receptacle_Amphenol_12401610E4-2A, symbol Connector:USB_C_Receptacle
- added JP1, JP2, JP3, JP4, JP5, JP6: SolderJumper_2_Open, Jumper:SolderJumper-2_P1.3mm_Open_Pad1.0x1.5mm, symbol Jumper:SolderJumper_2_Open
- added LED33, LED34, LED35, LED36, LED37, LED38, LED39, LED40, LED41, LED42, LED43, LED44, LED45, LED46, LED47, LED48, LED49, LED50, LED51, LED52, LED53, LED54, LED55, LED56, LED57, LED58, LED59, LED60, LED61, LED62, LED63, LED64: MX_SK6812MINI-E, lib:LED_MX_SK6812MINI-R, symbol marbastlib-mx:MX_SK6812MINI-E
- added R10: 10k, Resistor_SMD:R_0603_1608Metric, symbol Device:R
- added R11, R16, R9: 1k, Resistor_SMD:R_0603_1608Metric, symbol Device:R
- added R12, R13: 27.4, Resistor_SMD:R_0603_1608Metric, symbol Device:R
- added R14, R15: 5k1, Resistor_SMD:R_0603_1608Metric, symbol Device:R
- added SW3: BOOT, Button_Switch_SMD:SW_Push_1P1T_NO_Vertical_Wuerth_434133025816, symbol Switch:SW_Push
- added SW4: RESET, Button_Switch_SMD:SW_Push_1P1T_NO_Vertical_Wuerth_434133025816, symbol Switch:SW_Push
- added U40, U41, U42, U43, U44, U45, U46, U47, U48, U50, U51, U52, U53, U54, U55, U56, U57, U58, U59, U60, U61, U62, U63, U65, U66, U67, U68, U69, U70, U71, U77, U78: DRV5057A3, lib:DRV505x, symbol Sensor_Magnetic:DRV5055A3xDBZxQ1
- added U64: RP2040, Package_DFN_QFN:QFN-56-1EP_7x7mm_P0.4mm_EP3.2x3.2mm, symbol MCU_RaspberryPi:RP2040
- added U72: NCP1117-3.3_SOT223, Package_TO_SOT_SMD:SOT-223-3_TabPin2, symbol Regulator_Linear:NCP1117-3.3_SOT223
- added U73, U74, U75, U76: 74HC4051, Package_SO:TSSOP-16_4.4x5mm_P0.65mm, symbol 74xx:74HC4051
- added Y2: ECS-120-8-30-JGN-TR, Crystal:Crystal_SMD_5032-2Pin_5.0x3.2mm, symbol Device:Crystal
Connections:
- net +3.3V: now also JP2.2 (B), JP6.2 (B); no longer J1.1 (Pin_1), U10.2 (VCC)
- net +5V: now also C16.1, J4.A4 (VBUS), J4.A9 (VBUS), J4.B4 (VBUS), J4.B9 (VBUS), LED33.1 (VDD), LED34.1 (VDD), LED35.1 (VDD), LED36.1 (VDD), LED37.1 (VDD), LED38.1 (VDD), LED39.1 (VDD), LED40.1 (VDD), LED41.1 (VDD), LED42.1 (VDD), LED43.1 (VDD), LED44.1 (VDD), LED45.1 (VDD), LED46.1 (VDD), LED47.1 (VDD), LED48.1 (VDD), LED49.1 (VDD), LED50.1 (VDD), LED51.1 (VDD), LED52.1 (VDD), LED53.1 (VDD), LED54.1 (VDD), LED55.1 (VDD), LED56.1 (VDD), LED57.1 (VDD), LED58.1 (VDD), LED59.1 (VDD), LED60.1 (VDD), LED61.1 (VDD), LED62.1 (VDD), LED63.1 (VDD), LED64.1 (VDD), U72.3 (VI)
- net D_CS: now also JP4.1 (A)
- net D_DC: now also JP3.1 (A)
- net D_RST: now also U64.13 (GPIO10)
- net D_SDA: now also U64.12 (GPIO9)
- net GND: now also J2.SH (SHIELD), C11.2, C14.1, C15.2, C16.2, C17.1, C18.2, C19.1, C20.2, IC2.4 (GND), IC2.9 (EP), J4.A1 (GND), J4.A12 (GND), J4.B1 (GND), J4.B12 (GND), J4.SH (SHIELD), JP1.2 (B), JP4.2 (B), LED33.4 (VSS), LED34.4 (VSS), LED35.4 (VSS), LED36.4 (VSS), LED37.4 (VSS), LED38.4 (VSS), LED39.4 (VSS), LED40.4 (VSS), LED41.4 (VSS), LED42.4 (VSS), LED43.4 (VSS), LED44.4 (VSS), LED45.4 (VSS), LED46.4 (VSS), LED47.4 (VSS), LED48.4 (VSS), LED49.4 (VSS), LED50.4 (VSS), LED51.4 (VSS), LED52.4 (VSS), LED53.4 (VSS), LED54.4 (VSS), LED55.4 (VSS), LED56.4 (VSS), LED57.4 (VSS), LED58.4 (VSS), LED59.4 (VSS), LED60.4 (VSS), LED61.4 (VSS), LED62.4 (VSS), LED63.4 (VSS), LED64.4 (VSS), R14.2, R15.2, SW3.1, SW4.1, U40.3 (GND), U41.3 (GND), U42.3 (GND), U43.3 (GND), U44.3 (GND), U45.3 (GND), U46.3 (GND), U47.3 (GND), U48.3 (GND), U50.3 (GND), U51.3 (GND), U52.3 (GND), U53.3 (GND), U54.3 (GND), U55.3 (GND), U56.3 (GND), U57.3 (GND), U58.3 (GND), U59.3 (GND), U60.3 (GND), U61.3 (GND), U62.3 (GND), U63.3 (GND), U64.19 (TESTEN), U64.57 (GND), U65.3 (GND), U66.3 (GND), U67.3 (GND), U68.3 (GND), U69.3 (GND), U70.3 (GND), U71.3 (GND), U72.1 (GND), U73.7 (VEE), U73.8 (GND), U74.7 (VEE), U74.8 (GND), U75.7 (VEE), U75.8 (GND), U76.7 (VEE), U76.8 (GND), U77.3 (GND), U78.3 (GND); no longer U10.1 (GND)
- net USB_D+: now reaches J2.A6 (D+), J2.B6 (D+), R5.1
- net USB_D+: now also J4.A6 (D+), J4.B6 (D+), R13.1
- net USB_D-: now reaches J2.A7 (D-), J2.B7 (D-), R4.1
- net USB_D-: now also J4.A7 (D-), J4.B7 (D-), R12.1
- net SWD: now reaches J1.2 (Pin_2), U25.25 (SWD)
- net SWD: now also U64.25 (SWD)
- net SWCLK: now reaches J1.3 (Pin_3), U25.24 (SWCLK)
- net SWCLK: now also U64.24 (SWCLK)
- net D_SCL renamed D_RST_R
- net D_RST_R: now also U64.11 (GPIO8)
- new net: LED45.2 (DOUT), LED50.3 (DIN)
- new net: LED41.2 (DOUT), LED45.3 (DIN)
- new net: C14.2, C17.2, C19.2, U64.23 (DVDD), U64.45 (VREG_VOUT), U64.50 (DVDD)
- new net: U58.2 (OUT), U76.4 (A7)
- new net: U66.2 (OUT), U73.1 (A4)
- new net: U70.2 (OUT), U73.12 (A3)
- new net: U45.2 (OUT), U73.13 (A0)
- new net: U40.2 (OUT), U73.14 (A1)
- new net: U44.2 (OUT), U73.15 (A2)
- new net: U60.2 (OUT), U73.2 (A6)
- new net: U55.2 (OUT), U73.4 (A7)
- new net: U50.2 (OUT), U73.5 (A5)
- new net: U61.2 (OUT), U74.2 (A6)
- new net: C13.2, U64.20 (XIN)
- new net: R11.2, U64.21 (XOUT)
- new net: R16.2, U64.26 (RUN)
- new net: R12.2, U64.46 (USB_DM)
- new net: R13.2, U64.47 (USB_DP)
- new net: LED34.3 (DIN), LED35.2 (DOUT)
- new net: LED35.3 (DIN), LED40.2 (DOUT)
- new net: LED61.3 (DIN), LED63.2 (DOUT)
- new net: LED63.3 (DIN), LED64.2 (DOUT)
- new net: U41.2 (OUT), U74.14 (A1)
- new net: LED34.2 (DOUT), LED39.3 (DIN)
- new net: C13.1, Y2.2
- new net: LED57.3 (DIN), LED58.2 (DOUT)
- new net: LED53.2 (DOUT), LED58.3 (DIN)
- new net: LED59.3 (DIN), LED60.2 (DOUT)
- new net: LED55.2 (DOUT), LED60.3 (DIN)
- new net: LED44.3 (DIN), LED49.2 (DOUT)
- new net: LED49.3 (DIN), LED54.2 (DOUT)
- new net: LED38.3 (DIN), LED42.2 (DOUT)
- new net: LED42.3 (DIN), LED47.2 (DOUT)
- new net: C12.1, Y2.1
- new net: U68.2 (OUT), U75.1 (A4)
- new net: U75.12 (A3), U78.2 (OUT)
- new net: U47.2 (OUT), U75.13 (A0)
- new net: U42.2 (OUT), U75.14 (A1)
- new net: U59.2 (OUT), U75.15 (A2)
- new net: U62.2 (OUT), U75.2 (A6)
- new net: U57.2 (OUT), U75.4 (A7)
- new net: U52.2 (OUT), U75.5 (A5)
- new net: LED48.2 (DOUT), LED53.3 (DIN)
- new net: C12.2, R11.1
- new net: LED43.2 (DOUT), LED48.3 (DIN)
- new net: LED39.2 (DOUT), LED43.3 (DIN)
- new net: LED56.3 (DIN), LED61.2 (DOUT)
- new net: J4.A5 (CC1), R15.1
- new net: J4.B5 (CC2), R14.1
- new net: U54.2 (OUT), U74.15 (A2)
- new net: R9.1, SW3.2
- new net: U63.2 (OUT), U76.2 (A6)
- new net: R16.1, SW4.2
- new net: LED46.3 (DIN), LED51.2 (DOUT)
- new net: LED51.3 (DIN), LED56.2 (DOUT)
- new net: LED47.3 (DIN), LED52.2 (DOUT)
- new net: LED40.3 (DIN), LED44.2 (DOUT)
- new net: J1.1 (Pin_1), JP5.1 (A), JP6.1 (A)
- new net: U53.2 (OUT), U76.5 (A5)
- new net: LED54.3 (DIN), LED59.2 (DOUT)
- new net: LED33.3 (DIN), LED38.2 (DOUT)
- new net: LED36.2 (DOUT), LED41.3 (DIN)
- new net: U65.2 (OUT), U76.15 (A2)
- new net: LED50.2 (DOUT), LED55.3 (DIN)
- new net: U51.2 (OUT), U74.5 (A5)
- new net: U67.2 (OUT), U74.1 (A4)
- new net: U74.12 (A3), U77.2 (OUT)
- new net: U46.2 (OUT), U74.13 (A0)
- new net: U56.2 (OUT), U74.4 (A7)
- new net: LED36.3 (DIN), LED37.2 (DOUT)
- new net: U43.2 (OUT), U76.14 (A1)
- new net: LED37.3 (DIN), LED46.2 (DOUT)
- new net: U71.2 (OUT), U76.12 (A3)
- new net: LED62.2 (DOUT), LED64.3 (DIN)
- new net: LED52.3 (DIN), LED57.2 (DOUT)
- new net: U69.2 (OUT), U76.1 (A4)
- new net: U48.2 (OUT), U76.13 (A0)
- new net +3.3VR: C11.1, C15.1, C18.1, C20.1, IC2.8 (VCC), JP3.2 (B), JP5.2 (B), R10.2, U40.1 (VCC), U41.1 (VCC), U42.1 (VCC), U43.1 (VCC), U44.1 (VCC), U45.1 (VCC), U46.1 (VCC), U47.1 (VCC), U48.1 (VCC), U50.1 (VCC), U51.1 (VCC), U52.1 (VCC), U53.1 (VCC), U54.1 (VCC), U55.1 (VCC), U56.1 (VCC), U57.1 (VCC), U58.1 (VCC), U59.1 (VCC), U60.1 (VCC), U61.1 (VCC), U62.1 (VCC), U63.1 (VCC), U64.1 (IOVDD), U64.10 (IOVDD), U64.22 (IOVDD), U64.33 (IOVDD), U64.42 (IOVDD), U64.43 (ADC_AVDD), U64.44 (VREG_IN), U64.48 (USB_VDD), U64.49 (IOVDD), U65.1 (VCC), U66.1 (VCC), U67.1 (VCC), U68.1 (VCC), U69.1 (VCC), U70.1 (VCC), U71.1 (VCC), U72.2 (VO), U73.16 (VCC), U74.16 (VCC), U75.16 (VCC), U76.16 (VCC), U77.1 (VCC), U78.1 (VCC)
- new net D_CS_R: JP1.1 (A), U10.1 (GND), U64.8 (GPIO6)
- new net D_DC_R: JP2.1 (A), U10.2 (VCC), U64.9 (GPIO7)
- new net LED R: LED62.3 (DIN), U64.32 (GPIO21)
- new net MUX R E: U64.37 (GPIO25), U73.6 (~{E}), U74.6 (~{E}), U75.6 (~{E}), U76.6 (~{E})
- new net MUX R S0: U64.36 (GPIO24), U73.11 (S0), U74.11 (S0), U75.11 (S0), U76.11 (S0)
- new net MUX R S1: U64.35 (GPIO23), U73.10 (S1), U74.10 (S1), U75.10 (S1), U76.10 (S1)
- new net MUX R S2: U64.34 (GPIO22), U73.9 (S2), U74.9 (S2), U75.9 (S2), U76.9 (S2)
- new net MUX1R COM: U64.41 (GPIO29_ADC3), U73.3 (A)
- new net MUX2R COM: U64.40 (GPIO28_ADC2), U74.3 (A)
- new net MUX3R COM: U64.39 (GPIO27_ADC1), U75.3 (A)
- new net MUX4R COM: U64.38 (GPIO26_ADC0), U76.3 (A)
- new net QSPI_R_SCLK: IC2.6 (CLK), U64.52 (QSPI_SCLK)
- new net QSPI_R_SD0: IC2.5 (DI(IO0)), U64.53 (QSPI_SD0)
- new net QSPI_R_SD1: IC2.2 (DO(IO1)), U64.55 (QSPI_SD1)
- new net QSPI_R_SD2: IC2.3 (IO2), U64.54 (QSPI_SD2)
- new net QSPI_R_SD3: IC2.7 (IO3), U64.51 (QSPI_SD3)
- new net QSPI_R_SS: IC2.1 (~{CS}), R10.1, R9.2, U64.56 (QSPI_SS)
Other:
- moved on the sheet: C1, C10, C2, C3, C4, C5, C6, C7, C8, C9, IC1, J1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

Commit message: usb-c interconnects and expansion solder pads
Parts:
- added J5, J8: Conn_01x05_Socket, lib:TestPad_5pins, symbol Connector:Conn_01x05_Socket
- added J6, J7: USB_C_Interlink, Connector_USB:USB_C_Receptacle_Amphenol_12401610E4-2A, symbol Connector:USB_C_Receptacle
- added R17, R18, R19, R20: 56k, Resistor_SMD:R_0603_1608Metric, symbol Device:R
- J2, J4: value USB_C_Receptacle -> USB_C_To_Host
Connections:
- net +3.3V: now also J8.5 (Pin_5)
- net +3.3VR: now also J5.5 (Pin_5)
- net +5V: now also J5.4 (Pin_4), J6.A4 (VBUS), J6.A9 (VBUS), J6.B4 (VBUS), J6.B9 (VBUS), J7.A4 (VBUS), J7.A9 (VBUS), J7.B4 (VBUS), J7.B9 (VBUS), J8.4 (Pin_4), R17.1, R18.1, R19.1, R20.1
- net GND: now also J5.1 (Pin_1), J6.A1 (GND), J6.A12 (GND), J6.B1 (GND), J6.B12 (GND), J6.SH (SHIELD), J7.A1 (GND), J7.A12 (GND), J7.B1 (GND), J7.B12 (GND), J7.SH (SHIELD), J8.1 (Pin_1)
- net I2C ACC R SDA: now reaches U64.2 (GPIO0)
- net I2C ACC R SDA: now also J5.3 (Pin_3)
- net I2C R SDA: now reaches U64.27 (GPIO16)
- net I2C R SDA: now also J7.A7 (D-), J7.B7 (D-)
- net I2C R SDL: now reaches U64.28 (GPIO17)
- net I2C R SDL: now also J7.A6 (D+), J7.B6 (D+)
- net I2C ACC R SDL: now reaches U64.3 (GPIO1)
- net I2C ACC R SDL: now also J5.2 (Pin_2)
- net I2C ACC SDA: now reaches U25.2 (GPIO0)
- net I2C ACC SDA: now also J8.3 (Pin_3)
- net I2C SDA: now reaches U25.27 (GPIO16)
- net I2C SDA: now also J6.A7 (D-), J6.B7 (D-)
- net I2C SDL: now reaches U25.28 (GPIO17)
- net I2C SDL: now also J6.A6 (D+), J6.B6 (D+)
- net I2C ACC SDL: now reaches U25.3 (GPIO1)
- net I2C ACC SDL: now also J8.2 (Pin_2)
- new net: J6.B5 (CC2), R18.2
- new net: J7.B5 (CC2), R19.2
- new net: J6.A5 (CC1), R17.2
- new net: J7.A5 (CC1), R20.2
