File: woodox/woodox.kicad_sch (KiCad schematic)
At the start: 202 parts, among them IC1 W25Q16JVUXIQ_TR, IC2 W25Q16JVUXIQ_TR, J1 Conn_01x03_Female, J2 USB_C_To_Host, J4 USB_C_To_Host, J5 Conn_01x05_Socket, J6 USB_C_Interlink, J7 USB_C_Interlink, J8 Conn_01x05_Socket, SW1 BOOT, SW2 RESET, SW3 BOOT, SW4 RESET, U1 DRV5057A3, U10 OLED_256x64_I2C, U11 DRV5057A3, U12 DRV5057A3, U13 DRV5057A3, U14 DRV5057A3, U15 DRV5057A3, U16 DRV5057A3, U17 DRV5057A3, U18 DRV5057A3, U19 DRV5057A3, U2 DRV5057A3, U20 DRV5057A3, U21 DRV5057A3, U22 DRV5057A3, U23 DRV5057A3, U24 DRV5057A3, U25 RP2040, U26 DRV5057A3, U27 DRV5057A3, U28 DRV5057A3, U29 DRV5057A3, U3 DRV5057A3, U30 DRV5057A3, U31 DRV5057A3, U32 DRV5057A3, U33 NCP1117-3.3_SOT223, U34 74HC4051, U35 74HC4051, U36 74HC4051, U37 74HC4051, U38 DRV5057A3, U39 DRV5057A3, U4 DRV5057A3, U40 DRV5057A3, U41 DRV5057A3, U42 DRV5057A3, U43 DRV5057A3, U44 DRV5057A3, U45 DRV5057A3, U46 DRV5057A3, U47 DRV5057A3, U48 DRV5057A3, U5 DRV5057A3, U50 DRV5057A3, U51 DRV5057A3, U52 DRV5057A3, U53 DRV5057A3, U54 DRV5057A3, U55 DRV5057A3, U56 DRV5057A3, U57 DRV5057A3, U58 DRV5057A3, U59 DRV5057A3, U6 DRV5057A3, U60 DRV5057A3, U61 DRV5057A3, U62 DRV5057A3, U63 DRV5057A3, U64 RP2040, U65 DRV5057A3, U66 DRV5057A3, U67 DRV5057A3, U68 DRV5057A3, U69 DRV5057A3, U7 DRV5057A3, U70 DRV5057A3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

Commit message: rp2350 redesign
Parts:
- removed C1, C11, C17, C19, C7, C9: 0.1uF, Capacitor_SMD:C_0603_1608Metric, symbol Device:C_Small
- removed C12, C13, C2, C3: 27pF, Capacitor_SMD:C_0603_1608Metric, symbol Device:C_Small
- removed C14, C15, C18, C4, C5, C8: 1uF, Capacitor_SMD:C_0603_1608Metric, symbol Device:C_Small
- removed IC1, IC2: W25Q16JVUXIQ_TR, W25Q16JVUXIQ_TR:SON50P300X200X60-9N, symbol W25Q16JVUXIQ_TR:W25Q16JVUXIQ_TR
- removed JP5, JP6: SolderJumper_2_Open, Jumper:SolderJumper-2_P1.3mm_Open_Pad1.0x1.5mm, symbol Jumper:SolderJumper_2_Open
- removed R10: 10k, Resistor_SMD:R_0603_1608Metric, symbol Device:R
- removed R3, R8, R9: 1k, Resistor_SMD:R_0603_1608Metric, symbol Device:R
- removed R4, R5: 27.4, Resistor_SMD:R_0603_1608Metric, symbol Device:R
- removed U25, U64: RP2040, Package_DFN_QFN:QFN-56-1EP_7x7mm_P0.4mm_EP3.2x3.2mm, symbol MCU_RaspberryPi:RP2040
- removed Y1, Y2: ECS-120-8-30-JGN-TR, Crystal:Crystal_SMD_5032-2Pin_5.0x3.2mm, symbol Device:Crystal
- added C12, C13, C21, C22: 4.7u, RP2350_80QFN_minimal:C_0402_1005Metric_small_pads, symbol Device:C
- added C14, C17, C24, C25: 4.7u, Capacitor_SMD:C_0402_1005Metric, symbol Device:C
- added C15, C18, C19, C23, C26, C27, C32, C33, C34, C35, C36, C37, C38, C39, C4, C44, C45, C46, C47, C48, C49, C5, C50, C51: 100n, Capacitor_SMD:C_0402_1005Metric, symbol Device:C
- added C40, C41, C42, C43: 15p, Capacitor_SMD:C_0402_1005Metric, symbol Device:C
- added L2, L3: 3.3u, RP2350_80QFN_minimal:L_pol_2016, symbol Device:L
- added R21: 1k, Resistor_SMD:R_0402_1005Metric, symbol Device:R
- added R22, R26: 33, Resistor_SMD:R_0402_1005Metric, symbol Device:R
- added R23: 1k, Resistor_SMD:R_0603_1608Metric, symbol Device:R
- added R24, R25, R27, R28: 27, Resistor_SMD:R_0402_1005Metric, symbol Device:R
- added U25, U49: W25Q128JVP, Package_SON:WSON-8-1EP_6x5mm_P1.27mm_EP3.4x4.3mm, symbol Memory_Flash:W25Q128JVS
- added U64, U79: RP2350_80QFN, Package_DFN_QFN:QFN-80-1EP_10x10mm_P0.4mm_EP3.4x3.4mm_ThermalVias, symbol MCU_RaspberryPi_RP2350:RP2350_80QFN
- added Y2, Y3: ABM8-272-T3, Crystal:Crystal_SMD_3225-4Pin_3.2x2.5mm, symbol Device:Crystal_GND24
- C16, C20, R14, R15, R17, R18, R19, R20: KiLib_Generator (none) -> SMD_2terminal_chip_molded
- J1: footprint Connector_PinHeader_2.54mm:PinHeader_1x04_P2.54mm_Vertical -> Connector_PinHeader_2.54mm:PinHeader_1x03_P2.54mm_Vertical; symbol Connector:Conn_01x04_Female -> Connector:Conn_01x03_Socket
- R1, R16: MPN RCC06031K00FKEA -> (none)
- R11: value 1k -> DNF; MPN RCC06031K00FKEA -> ERJ-3EKF1002V; now not fitted
- R12: value 27.4 -> 1k; footprint Resistor_SMD:R_0603_1608Metric -> Resistor_SMD:R_0402_1005Metric; MPN CRCW060327R4FKEB -> (none)
- R13: value 27.4 -> DNF; MPN CRCW060327R4FKEB -> ERJ-3EKF1002V; now not fitted
- R2: value 10k -> 1k; MPN ERJ-3EKF1002V -> (none)
- SW1, SW3: value BOOT -> SW_Push; MPN 95C06B2GWRT -> (none)
- SW2, SW4: value RESET -> SW_Push; MPN 95C06B2GWRT -> (none)
- U73, U74, U75, U76: KiLib_Generator (none) -> package/gullwing
Connections:
- net +3.3V: now also R11.2, C12.1, C18.1, C19.1, C32.1, C33.1, C34.1, C35.1, C36.1, C37.1, C38.1, C4.1, R22.1, U25.8 (VCC), U64.15 (IOVDD), U64.24 (IOVDD), U64.29 (IOVDD), U64.41 (IOVDD), U64.5 (IOVDD), U64.50 (IOVDD), U64.59 (ADC_AVDD), U64.60 (IOVDD), U64.64 (VREG_VIN), U64.68 (USB_OTP_VDD), U64.69 (QSPI_IOVDD), U64.76 (IOVDD); no longer R2.2
- net +3.3VR: now also R13.2, C21.1, C26.1, C27.1, C45.1, C46.1, C47.1, C48.1, C49.1, C5.1, C50.1, C51.1, R26.1, U49.8 (VCC), U79.15 (IOVDD), U79.24 (IOVDD), U79.29 (IOVDD), U79.41 (IOVDD), U79.5 (IOVDD), U79.50 (IOVDD), U79.59 (ADC_AVDD), U79.60 (IOVDD), U79.64 (VREG_VIN), U79.68 (USB_OTP_VDD), U79.69 (QSPI_IOVDD), U79.76 (IOVDD)
- net D_CS: now also U64.43 (GPIO34)
- net D_CS_R: now also U79.43 (GPIO34)
- net D_DC: now also U64.44 (GPIO35)
- net D_DC_R: now also U79.44 (GPIO35)
- net D_RST: now also U64.45 (GPIO36), U79.47 (GPIO38)
- net D_RST_R: now also U64.47 (GPIO38), U79.45 (GPIO36)
- net D_SDA: now also U64.46 (GPIO37), U79.46 (GPIO37)
- net GND: now also J1.1 (Pin_1), R16.2, C12.2, C13.2, C14.2, C15.2, C17.2, C18.2, C19.2, C21.2, C22.2, C23.2, C24.2, C25.2, C26.2, C27.2, C32.2, C33.2, C34.2, C35.2, C36.2, C37.2, C38.2, C39.2, C4.2, C40.2, C41.2, C42.2, C43.2, C44.2, C45.2, C46.2, C47.2, C48.2, C49.2, C5.2, C50.2, C51.2, R23.2, U25.4 (GND), U49.4 (GND), U64.62 (VREG_PGND), U64.81 (GND), U79.62 (VREG_PGND), U79.81 (GND), Y2.2 (G), Y2.4 (G), Y3.2 (G), Y3.4 (G); no longer J1.4 (Pin_4), SW2.1, SW4.1
- net I2C ACC R SDA: no longer J5.3 (Pin_3)
- net I2C ACC R SDL: no longer J5.2 (Pin_2)
- net I2C ACC SDA: now also U64.3 (GPIO6)
- net I2C ACC SDL: now also U64.4 (GPIO7)
- net I2C R SDA: now also U79.1 (GPIO4)
- net I2C R SDL: now also U79.2 (GPIO5)
- net I2C SDA: now also U64.1 (GPIO4)
- net I2C SDL: now also U64.2 (GPIO5)
- net LED: now also U64.42 (GPIO33)
- net LED R: now also U79.42 (GPIO33)
- net MUX E: now also U64.40 (GPIO32)
- net MUX R E: now also U79.40 (GPIO32)
- net MUX R S0: now also U79.39 (GPIO31)
- net MUX R S1: now also U79.38 (GPIO30)
- net MUX R S2: now also U79.37 (GPIO29)
- net MUX S0: now also U64.39 (GPIO31)
- net MUX S1: now also U64.38 (GPIO30)
- net MUX S2: now also U64.37 (GPIO29)
- net MUX1 COM: now also U64.55 (GPIO44_ADC4)
- net MUX1R COM: now also U79.55 (GPIO44_ADC4)
- net MUX2 COM: now also U64.54 (GPIO43_ADC3)
- net MUX2R COM: now also U79.54 (GPIO43_ADC3)
- net MUX3 COM: now also U64.53 (GPIO42_ADC2)
- net MUX3R COM: now also U79.53 (GPIO42_ADC2)
- net MUX4 COM: now also U64.52 (GPIO41_ADC1)
- net MUX4R COM: now also U79.52 (GPIO41_ADC1)
- net QSPI_R_SCLK: now also U49.6 (CLK), U79.71 (QSPI_SCLK)
- net QSPI_R_SD0: now also U49.5 (DI(IO0)), U79.72 (QSPI_SD0)
- net QSPI_R_SD1: now also U49.2 (DO(IO1)), U79.74 (QSPI_SD1)
- net QSPI_R_SD2: now also U49.3 (IO2), U79.73 (QSPI_SD2)
- net QSPI_R_SD3: now also U49.7 (IO3), U79.70 (QSPI_SD3)
- net QSPI_R_SS: now also R13.1, R2.1, U49.1 (~{CS}), U79.75 (QSPI_SS)
- net QSPI_SCLK: now also U25.6 (CLK), U64.71 (QSPI_SCLK)
- net QSPI_SD0: now also U25.5 (DI(IO0)), U64.72 (QSPI_SD0)
- net QSPI_SD1: now also U25.2 (DO(IO1)), U64.74 (QSPI_SD1)
- net QSPI_SD2: now also U25.3 (IO2), U64.73 (QSPI_SD2)
- net QSPI_SD3: now also U25.7 (IO3), U64.70 (QSPI_SD3)
- net QSPI_SS: now also R1.1, R11.1, U25.1 (~{CS}), U64.75 (QSPI_SS); no longer R1.2, R2.1
- net SWCLK: now also U64.33 (SWCLK), U79.33 (SWCLK)
- net SWD: now also U64.34 (SWD), U79.34 (SWD)
- net USB_D+: now also R24.1, R27.1; no longer R13.1
- net USB_D-: now also R25.1, R28.1; no longer R12.1
- net at R12.2: now also C41.1, Y2.3
- net RUN: now reaches SW2.2
- net RUN: now also U64.35 (RUN)
- net ~{USB_BOOT_R}: now reaches SW3.2
- net ~{USB_BOOT_R}: now also R2.2
- net at R16.1: now also SW2.1; no longer SW4.2
- net ~{USB_BOOT}: now reaches SW1.2
- net ~{USB_BOOT}: now also R1.2; no longer R1.1
- new net: C40.1, U64.30 (XIN), Y2.1
- new net: R12.1, U64.31 (XOUT)
- new net: R25.2, U64.66 (USB_DM)
- new net: R24.2, U64.67 (USB_DP)
- new net: R23.1, SW4.1
- new net: C42.1, U79.30 (XIN), Y3.1
- new net: C43.1, R21.2, Y3.3
- new net: R28.2, U79.66 (USB_DM)
- new net: SW4.2, U79.35 (RUN)
- new net: R27.2, U79.67 (USB_DP)
- new net: R21.1, U79.31 (XOUT)
- new net +1V1: C13.1, C15.1, C17.1, C22.1, C23.1, C25.1, C39.1, C44.1, L2.1, L3.1, U64.10 (DVDD), U64.32 (DVDD), U64.51 (DVDD), U64.65 (VREG_FB), U79.10 (DVDD), U79.32 (DVDD), U79.51 (DVDD), U79.65 (VREG_FB)
- new net I2C R ACC SDA: J5.3 (Pin_3), U79.3 (GPIO6)
- new net I2C R ACC SDL: J5.2 (Pin_2), U79.4 (GPIO7)
- new net VREG_AVDD: C14.1, R22.2, U64.61 (VREG_AVDD)
- new net VREG_AVDD_R: C24.1, R26.2, U79.61 (VREG_AVDD)
- new net VREG_LX: L2.2, U64.63 (VREG_LX)
- new net VREG_LX_R: L3.2, U79.63 (VREG_LX)
Other:
- note added: "12MHz Crystal"
- note added: "Make sure R7 and R8 are close to RP2350"
- note added: "Primary Flash"
- moved on the sheet: J5, J6, J7, J8, LED1, LED10, LED11, LED12, LED13, LED14, LED15, LED16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

Commit message: fix lints
Parts:
- U64, U79: footprint Package_DFN_QFN:QFN-80-1EP_10x10mm_P0.4mm_EP3.4x3.4mm_ThermalVias -> RP2350_80QFN_minimal:RP2350-QFN-80-1EP_10x10_P0.4mm_EP3.4x3.4mm_ThermalVias
Changed lines of the file:
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@@
 			)
 		)
-		(property "Footprint" "Package_DFN_QFN:QFN-80-1EP_10x10mm_P0.4mm_EP3.4x3.4mm_ThermalVias"
+		(property "Footprint" "RP2350_80QFN_minimal:RP2350-QFN-80-1EP_10x10_P0.4mm_EP3.4x3.4mm_ThermalVias"
 			(at 137.16 275.59 0)
 			(hide yes)
@@
 			)
 		)
-		(property "Footprint" "Package_DFN_QFN:QFN-80-1EP_10x10mm_P0.4mm_EP3.4x3.4mm_ThermalVias"
+		(property "Footprint" "RP2350_80QFN_minimal:RP2350-QFN-80-1EP_10x10_P0.4mm_EP3.4x3.4mm_ThermalVias"
 			(at 425.45 281.94 0)
 			(hide yes)
