File: woodox/woodox.kicad_sch (KiCad schematic)
At the start: 224 parts, among them J1 Conn_01x03_Female, J2 USB_C_To_Host, J4 USB_C_To_Host, J5 Conn_01x05_Socket, J6 USB_C_Interlink, J7 USB_C_Interlink, J8 Conn_01x05_Socket, SW1 SW_Push, SW2 SW_Push, SW3 SW_Push, SW4 SW_Push, U1 DRV5057A3, U10 OLED_256x64_I2C, U11 DRV5057A3, U12 DRV5057A3, U13 DRV5057A3, U14 DRV5057A3, U15 DRV5057A3, U16 DRV5057A3, U17 DRV5057A3, U18 DRV5057A3, U19 DRV5057A3, U2 DRV5057A3, U20 DRV5057A3, U21 DRV5057A3, U22 DRV5057A3, U23 DRV5057A3, U24 DRV5057A3, U25 W25Q128JVP, U26 DRV5057A3, U27 DRV5057A3, U28 DRV5057A3, U29 DRV5057A3, U3 DRV5057A3, U30 DRV5057A3, U31 DRV5057A3, U32 DRV5057A3, U33 NCP1117-3.3_SOT223, U34 74HC4051, U35 74HC4051, U36 74HC4051, U37 74HC4051, U38 DRV5057A3, U39 DRV5057A3, U4 DRV5057A3, U40 DRV5057A3, U41 DRV5057A3, U42 DRV5057A3, U43 DRV5057A3, U44 DRV5057A3, U45 DRV5057A3, U46 DRV5057A3, U47 DRV5057A3, U48 DRV5057A3, U49 W25Q128JVP, U5 DRV5057A3, U50 DRV5057A3, U51 DRV5057A3, U52 DRV5057A3, U53 DRV5057A3, U54 DRV5057A3, U55 DRV5057A3, U56 DRV5057A3, U57 DRV5057A3, U58 DRV5057A3, U59 DRV5057A3, U6 DRV5057A3, U60 DRV5057A3, U61 DRV5057A3, U62 DRV5057A3, U63 DRV5057A3, U64 RP2350_80QFN, U65 DRV5057A3, U66 DRV5057A3, U67 DRV5057A3, U68 DRV5057A3, U69 DRV5057A3, U7 DRV5057A3, U70 DRV5057A3, U71 DRV5057A3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

Commit message: mounting holes
Parts:
- added J10, J11, J12, J9: Conn_01x01, MountingHole:MountingHole_3.2mm_M3_DIN965_Pad, symbol Connector_Generic:Conn_01x01
- added J3: Conn_01x03_Female, lib:TestPad_3pins, symbol Connector:Conn_01x03_Socket
- added JP5, JP6, JP7, JP8: SolderJumper_2_Open, Jumper:SolderJumper-2_P1.3mm_Open_Pad1.0x1.5mm, symbol Jumper:SolderJumper_2_Open
- J1: footprint Connector_PinHeader_2.54mm:PinHeader_1x03_P2.54mm_Vertical -> lib:TestPad_3pins
Connections:
- net +3.3V: now also JP7.2 (B)
- net +3.3VR: now also JP6.2 (B)
- net GND: now also J10.1 (Pin_1), J11.1 (Pin_1), J12.1 (Pin_1), J3.1 (Pin_1), J9.1 (Pin_1), JP5.2 (B), JP8.2 (B)
- net SWCLK: now also J3.3 (Pin_3)
- net SWD: now also J3.2 (Pin_2)
- net at U64.6 (GPIO8): now also JP7.1 (A), JP8.1 (A)
- net at U79.6 (GPIO8): now also JP5.1 (A), JP6.1 (A)

Commit message: idk
Parts:
- C10, C16, C20, C6: footprint Capacitor_SMD:C_0603_1608Metric -> Capacitor_SMD:C_0402_1005Metric; IPN (none) -> CAP-000021
- C12, C13, C14, C17, C21, C22, C24, C25: IPN (none) -> CAP-000024
- C15, C18, C19, C23, C26, C27, C32, C33, C34, C35, C36, C37, C38, C39, C4, C44, C45, C46, C47, C48, C49, C5, C50, C51: IPN (none) -> CAP-000025
- C40, C41, C42, C43: IPN (none) -> CAP-000069
- J1, J10, J11, J12, J3, J5, J8, J9: now left out of the parts list
- J2, J4, J6, J7: IPN (none) -> CON-000041
- L2, L3: IPN (none) -> IND-000067; MPN (none) -> AOTA-B201610S3R3-101-T
- LED1, LED10, LED11, LED12, LED13, LED14, LED15, LED16, LED17, LED18, LED19, LED2, LED20, LED21, LED22, LED23, LED24, LED25, LED26, LED27, LED28, LED29, LED3, LED30, LED31, LED32, LED33, LED34, LED35, LED36, LED37, LED38, LED39, LED4, LED40, LED41, LED42, LED43, LED44, LED45, LED46, LED47, LED48, LED49, LED5, LED50, LED51, LED52, LED53, LED54, LED55, LED56, LED57, LED58, LED59, LED6, LED60, LED61, LED62, LED63, LED64, LED7, LED8, LED9: IPN (none) -> DIO-000012
- R1, R16, R2, R23: footprint Resistor_SMD:R_0603_1608Metric -> Resistor_SMD:R_0402_1005Metric; IPN (none) -> RES-000011
- R11, R13: footprint Resistor_SMD:R_0603_1608Metric -> Resistor_SMD:R_0402_1005Metric
- R12, R21: IPN (none) -> RES-000011
- R14, R15, R6, R7: footprint Resistor_SMD:R_0603_1608Metric -> Resistor_SMD:R_0402_1005Metric; IPN (none) -> RES-000015
- R17, R18, R19, R20: footprint Resistor_SMD:R_0603_1608Metric -> Resistor_SMD:R_0402_1005Metric; IPN (none) -> RES-000072
- R22, R26: IPN (none) -> RES-000071
- R24, R25, R27, R28: IPN (none) -> RES-000070
- SW1, SW2, SW3, SW4: IPN (none) -> MEC-000040
- U1, U11, U12, U13, U14, U15, U16, U17, U18, U19, U2, U20, U21, U22, U23, U24, U26, U27, U28, U29, U3, U30, U31, U32, U38, U39, U4, U40, U41, U42, U43, U44, U45, U46, U47, U48, U5, U50, U51, U52, U53, U54, U55, U56, U57, U58, U59, U6, U60, U61, U62, U63, U65, U66, U67, U68, U69, U7, U70, U71, U77, U78, U8, U9: IPN (none) -> ICS-000049
- U10: IPN (none) -> MIS-000056
- U25, U49: IPN (none) -> ICS-000065
- U33, U72: IPN (none) -> PWR-000043
- U34, U35, U36, U37, U73, U74, U75, U76: IPN (none) -> ICS-000064; MPN 74HC4051 -> CD74HC4051PWR
- U64, U79: IPN (none) -> ICS-000063
- Y2, Y3: IPN (none) -> CLK-000062
Other:
- moved on the sheet: J5, J6, J7, J8, R17, R18, R19, R20
